Commit message: Modified drive mode
Signed-off-by: Wonho Yun <ywh@robotis.com>

File: ffw_description/ros2_control/ffw_follower_with_rh_system.ros2_control.xacro (robot description, xacro)
@@ -124,64 +124,4 @@
           <state_interface name="velocity"/>
       </joint>
-      <joint name="arm_l_joint1">
-          <command_interface name="position"/>
-          <state_interface name="position">
-          </state_interface>
-          <state_interface name="velocity"/>
-      </joint>
-      <joint name="arm_l_joint2">
-          <command_interface name="position"/>
-          <state_interface name="position">
-          </state_interface>
-          <state_interface name="velocity"/>
-      </joint>
-      <joint name="arm_l_joint3">
-          <command_interface name="position"/>
-          <state_interface name="position">
-          </state_interface>
-          <state_interface name="velocity"/>
-      </joint>
-      <joint name="arm_l_joint4">
-          <command_interface name="position"/>
-          <state_interface name="position">
-          </state_interface>
-          <state_interface name="velocity"/>
-      </joint>
-      <joint name="arm_l_joint5">
-          <command_interface name="position"/>
-          <state_interface name="position">
-          </state_interface>
-          <state_interface name="velocity"/>
-      </joint>
-      <joint name="arm_l_joint6">
-          <command_interface name="position"/>
-          <state_interface name="position">
-          </state_interface>
-          <state_interface name="velocity"/>
-      </joint>
-      <joint name="arm_l_joint7">
-          <command_interface name="position"/>
-          <state_interface name="position">
-          </state_interface>
-          <state_interface name="velocity"/>
-      </joint>
-      <joint name="neck_joint1">
-          <command_interface name="position"/>
-          <state_interface name="position">
-          </state_interface>
-          <state_interface name="velocity"/>
-      </joint>
-      <joint name="neck_joint2">
-          <command_interface name="position"/>
-          <state_interface name="position">
-          </state_interface>
-          <state_interface name="velocity"/>
-      </joint>
-      <joint name="linear_joint">
-          <command_interface name="position"/>
-          <state_interface name="position">
-          </state_interface>
-          <state_interface name="velocity"/>
-      </joint>
       <joint name="r_rh_r1_joint">
         <command_interface name="position"/>
@@ -192,34 +132,46 @@
         <state_interface name="hardware_state"/>
       </joint>
-<!--
-      <xacro:if value="$(arg use_sim)">
-        <joint name="r_rh_r2">
-          <param name="mimic">r_rh_r1_joint</param>
-          <param name="multiplier">1.0</param>
-          <state_interface name="position"/>
-          <state_interface name="velocity"/>
-          <state_interface name="effort"/>
-          <state_interface name="torque_enable"/>
-          <state_interface name="hardware_state"/>
-        </joint>
-        <joint name="r_rh_l1">
-          <param name="mimic">r_rh_r1_joint</param>
-          <param name="multiplier">1.0</param>
-          <state_interface name="position"/>
-          <state_interface name="velocity"/>
-          <state_interface name="effort"/>
-          <state_interface name="torque_enable"/>
-          <state_interface name="hardware_state"/>
-        </joint>
-        <joint name="r_rh_l2">
-          <param name="mimic">r_rh_r1_joint</param>
-          <param name="multiplier">1.0</param>
-          <state_interface name="position"/>
-          <state_interface name="velocity"/>
-          <state_interface name="effort"/>
-          <state_interface name="torque_enable"/>
-          <state_interface name="hardware_state"/>
-        </joint>
-      </xacro:if> -->
+      <joint name="arm_l_joint1">
+          <command_interface name="position"/>
+          <state_interface name="position">
+          </state_interface>
+          <state_interface name="velocity"/>
+      </joint>
+      <joint name="arm_l_joint2">
+          <command_interface name="position"/>
+          <state_interface name="position">
+          </state_interface>
+          <state_interface name="velocity"/>
+      </joint>
+      <joint name="arm_l_joint3">
+          <command_interface name="position"/>
+          <state_interface name="position">
+          </state_interface>
+          <state_interface name="velocity"/>
+      </joint>
+      <joint name="arm_l_joint4">
+          <command_interface name="position"/>
+          <state_interface name="position">
+          </state_interface>
+          <state_interface name="velocity"/>
+      </joint>
+      <joint name="arm_l_joint5">
+          <command_interface name="position"/>
+          <state_interface name="position">
+          </state_interface>
+          <state_interface name="velocity"/>
+      </joint>
+      <joint name="arm_l_joint6">
+          <command_interface name="position"/>
+          <state_interface name="position">
+          </state_interface>
+          <state_interface name="velocity"/>
+      </joint>
+      <joint name="arm_l_joint7">
+          <command_interface name="position"/>
+          <state_interface name="position">
+          </state_interface>
+          <state_interface name="velocity"/>
+      </joint>
       <joint name="l_rh_r1_joint">
         <command_interface name="position"/>
@@ -230,34 +182,22 @@
         <state_interface name="hardware_state"/>
       </joint>
-<!--
-      <xacro:if value="$(arg use_sim)">
-        <joint name="l_rh_r2">
-          <param name="mimic">l_rh_r1_joint</param>
-          <param name="multiplier">1</param>
-          <state_interface name="position"/>
-          <state_interface name="velocity"/>
-          <state_interface name="effort"/>
-          <state_interface name="torque_enable"/>
-          <state_interface name="hardware_state"/>
-        </joint>
-        <joint name="l_rh_l1">
-          <param name="mimic">l_rh_r1_joint</param>
-          <param name="multiplier">1</param>
-          <state_interface name="position"/>
-          <state_interface name="velocity"/>
-          <state_interface name="effort"/>
-          <state_interface name="torque_enable"/>
-          <state_interface name="hardware_state"/>
-        </joint>
-        <joint name="l_rh_l2">
-          <param name="mimic">l_rh_r1_joint</param>
-          <param name="multiplier">1</param>
-          <state_interface name="position"/>
-          <state_interface name="velocity"/>
-          <state_interface name="effort"/>
-          <state_interface name="torque_enable"/>
-          <state_interface name="hardware_state"/>
-        </joint>
-      </xacro:if> -->
+      <joint name="neck_joint1">
+          <command_interface name="position"/>
+          <state_interface name="position">
+          </state_interface>
+          <state_interface name="velocity"/>
+      </joint>
+      <joint name="neck_joint2">
+          <command_interface name="position"/>
+          <state_interface name="position">
+          </state_interface>
+          <state_interface name="velocity"/>
+      </joint>
+      <joint name="linear_joint">
+          <command_interface name="position"/>
+          <state_interface name="position">
+          </state_interface>
+          <state_interface name="velocity"/>
+      </joint>
       <!-- RIGHT ARM -->
       <gpio name="dxl1">

File: ffw_description/ros2_control/ffw_leader_right_with_rh_system.ros2_control.xacro (robot description, xacro)
@@ -185,5 +185,5 @@
         <state_interface name="Torque Enable"/>
         <state_interface name="Present Input Voltage"/>
-        <param name="Drive Mode">0</param>
+        <param name="Drive Mode">1</param>
         <param name="Operating Mode">3</param>
         <param name="Return Delay Time">0</param>
