Commit message: Added low speed
Signed-off-by: Wonho Yun <ywh@robotis.com>

File: ffw_description/ros2_control/ffw_follower_with_rh_low_speed_system.ros2_control.xacro (robot description, xacro)
@@ -214,6 +214,6 @@
         <param name="Velocity Limit">2020</param>
         <param name="Acceleration Limit">20200</param>
-        <param name="Profile Velocity">2020</param>
-        <param name="Profile Acceleration">161</param>
+        <param name="Profile Velocity">804</param>
+        <param name="Profile Acceleration">40</param>
         <param name="Max Position Limit">131072</param>
         <param name="Min Position Limit">-131072</param>
@@ -235,6 +235,6 @@
         <param name="Velocity Limit">2020</param>
         <param name="Acceleration Limit">20200</param>
-        <param name="Profile Velocity">2020</param>
-        <param name="Profile Acceleration">161</param>
+        <param name="Profile Velocity">804</param>
+        <param name="Profile Acceleration">40</param>
         <param name="Max Position Limit">131072</param>
         <param name="Min Position Limit">0</param>
@@ -256,6 +256,6 @@
         <param name="Velocity Limit">2020</param>
         <param name="Acceleration Limit">20200</param>
-        <param name="Profile Velocity">2020</param>
-        <param name="Profile Acceleration">161</param>
+        <param name="Profile Velocity">804</param>
+        <param name="Profile Acceleration">40</param>
         <param name="Max Position Limit">262144</param>
         <param name="Min Position Limit">-262144</param>
@@ -277,6 +277,6 @@
         <param name="Velocity Limit">2020</param>
         <param name="Acceleration Limit">20200</param>
-        <param name="Profile Velocity">2020</param>
-        <param name="Profile Acceleration">161</param>
+        <param name="Profile Velocity">804</param>
+        <param name="Profile Acceleration">40</param>
         <param name="Max Position Limit">131072</param>
         <param name="Min Position Limit">-131072</param>
@@ -298,6 +298,6 @@
         <param name="Velocity Limit">2020</param>
         <param name="Acceleration Limit">20200</param>
-        <param name="Profile Velocity">2020</param>
-        <param name="Profile Acceleration">161</param>
+        <param name="Profile Velocity">804</param>
+        <param name="Profile Acceleration">40</param>
         <param name="Max Position Limit">262144</param>
         <param name="Min Position Limit">-262144</param>
@@ -319,6 +319,6 @@
         <param name="Velocity Limit">2020</param>
         <param name="Acceleration Limit">20200</param>
-        <param name="Profile Velocity">2020</param>
-        <param name="Profile Acceleration">161</param>
+        <param name="Profile Velocity">804</param>
+        <param name="Profile Acceleration">40</param>
         <param name="Max Position Limit">131072</param>
         <param name="Min Position Limit">-131072</param>
@@ -338,6 +338,6 @@
         <param name="Operating Mode">3</param>
         <param name="Return Delay Time">0</param>
-        <param name="Profile Velocity">2020</param>
-        <param name="Profile Acceleration">161</param>
+        <param name="Profile Velocity">804</param>
+        <param name="Profile Acceleration">40</param>
         <param name="Max Position Limit">101249</param>
         <param name="Min Position Limit">-101249</param>
@@ -369,6 +369,6 @@
         <param name="Velocity Limit">2020</param>
         <param name="Acceleration Limit">20200</param>
-        <param name="Profile Velocity">2020</param>
-        <param name="Profile Acceleration">161</param>
+        <param name="Profile Velocity">804</param>
+        <param name="Profile Acceleration">40</param>
         <param name="Max Position Limit">131072</param>
         <param name="Min Position Limit">-131072</param>
@@ -390,6 +390,6 @@
         <param name="Velocity Limit">2020</param>
         <param name="Acceleration Limit">20200</param>
-        <param name="Profile Velocity">2020</param>
-        <param name="Profile Acceleration">161</param>
+        <param name="Profile Velocity">804</param>
+        <param name="Profile Acceleration">40</param>
         <param name="Max Position Limit">131072</param>
         <param name="Min Position Limit">0</param>
@@ -411,6 +411,6 @@
         <param name="Velocity Limit">2020</param>
         <param name="Acceleration Limit">20200</param>
-        <param name="Profile Velocity">2020</param>
-        <param name="Profile Acceleration">161</param>
+        <param name="Profile Velocity">804</param>
+        <param name="Profile Acceleration">40</param>
         <param name="Max Position Limit">262144</param>
         <param name="Min Position Limit">-262144</param>
@@ -432,6 +432,6 @@
         <param name="Velocity Limit">2020</param>
         <param name="Acceleration Limit">20200</param>
-        <param name="Profile Velocity">2020</param>
-        <param name="Profile Acceleration">161</param>
+        <param name="Profile Velocity">804</param>
+        <param name="Profile Acceleration">40</param>
         <param name="Max Position Limit">131072</param>
         <param name="Min Position Limit">-131072</param>
@@ -453,6 +453,6 @@
         <param name="Velocity Limit">2020</param>
         <param name="Acceleration Limit">20200</param>
-        <param name="Profile Velocity">2020</param>
-        <param name="Profile Acceleration">161</param>
+        <param name="Profile Velocity">804</param>
+        <param name="Profile Acceleration">40</param>
         <param name="Max Position Limit">262144</param>
         <param name="Min Position Limit">-262144</param>
@@ -474,6 +474,6 @@
         <param name="Velocity Limit">2020</param>
         <param name="Acceleration Limit">20200</param>
-        <param name="Profile Velocity">2020</param>
-        <param name="Profile Acceleration">161</param>
+        <param name="Profile Velocity">804</param>
+        <param name="Profile Acceleration">40</param>
         <param name="Max Position Limit">131072</param>
         <param name="Min Position Limit">-131072</param>
@@ -493,6 +493,6 @@
         <param name="Operating Mode">3</param>
         <param name="Return Delay Time">0</param>
-        <param name="Profile Velocity">2020</param>
-        <param name="Profile Acceleration">161</param>
+        <param name="Profile Velocity">804</param>
+        <param name="Profile Acceleration">40</param>
         <param name="Max Position Limit">101249</param>
         <param name="Min Position Limit">-101249</param>

File: ffw_description/urdf/follower/ffw_follower_with_rh.urdf.xacro (robot description, xacro)
@@ -21,5 +21,5 @@
   </joint>
   <joint name="left_hand_fixed" type="fixed">
-    <origin xyz="0 0 -0.05" rpy="0 3.14 0"/>
+    <origin xyz="0 0 -0.05" rpy="0 3.14 -1.57"/>
     <parent link="arm_l_link7"/>
     <axis xyz="0 0 0"/>
@@ -27,5 +27,5 @@
   </joint>
   <joint name="right_hand_fixed" type="fixed">
-    <origin xyz="0 0 -0.05" rpy="0 3.14 0"/>
+    <origin xyz="0 0 -0.05" rpy="0 3.14 1.57"/>
     <parent link="arm_r_link7"/>
     <axis xyz="0 0 0"/>

File: ffw_description/urdf/follower/ffw_follower_with_rh_low_speed.urdf.xacro (robot description, xacro)
@@ -7,8 +7,10 @@
   <xacro:include filename="$(find ffw_description)/urdf/follower/ffw_follower_body.urdf.xacro" />
   <!-- Import control_xacro -->
-  <xacro:include filename="$(find ffw_description)/ros2_control/ffw_follower_system_only_left.ros2_control.xacro" />
-  <xacro:include filename="$(find ffw_description)/gazebo/ffw_follower.gazebo.xacro" />
-  <xacro:include filename="$(find ffw_description)/urdf/urdf_left_12_20.xacro" />
-  <xacro:include filename="$(find ffw_description)/urdf/urdf_right_12_20.xacro" />
+  <xacro:include filename="$(find ffw_description)/ros2_control/ffw_follower_with_rh_low_speed_system.ros2_control.xacro" />
+  <xacro:include filename="$(find ffw_description)/gazebo/ffw_follower_with_rh.gazebo.xacro" />
+  <xacro:include filename="$(find ffw_description)/urdf/left_rh_p12_rn_a.urdf.xacro" />
+  <xacro:include filename="$(find ffw_description)/urdf/right_rh_p12_rn_a.urdf.xacro" />
+<xacro:l_rh_p12_rn_a/>
+<xacro:r_rh_p12_rn_a/>
   <!-- World -->
   <link name="world"/>
@@ -19,14 +21,14 @@
   </joint>
   <joint name="left_hand_fixed" type="fixed">
-    <origin xyz="0 0 -0.05" rpy="0 0 0"/>
+    <origin xyz="0 0 -0.05" rpy="0 3.14 -1.57"/>
     <parent link="arm_l_link7"/>
     <axis xyz="0 0 0"/>
-    <child link="base_link_left_hand"/>
+    <child link="l_rh_p12_rn_base"/>
   </joint>
   <joint name="right_hand_fixed" type="fixed">
-    <origin xyz="0 0 -0.05" rpy="0 0 0"/>
+    <origin xyz="0 0 -0.05" rpy="0 3.14 1.57"/>
     <parent link="arm_r_link7"/>
     <axis xyz="0 0 0"/>
-    <child link="base_link_right_hand"/>
+    <child link="r_rh_p12_rn_base"/>
   </joint>
   <xacro:ffw_follower_system
