Commit message: Modified low speed version
Signed-off-by: Wonho Yun <ywh@robotis.com>

File: ffw_description/ros2_control/ffw_follower_with_rh_low_speed_system.ros2_control.xacro (robot description, xacro)
@@ -1,561 +1,577 @@
-<?xml version="1.0"?>
-<robot xmlns:xacro="http://www.ros.org/wiki/xacro">
-  <xacro:macro name="ffw_follower_system" params="use_sim:=^|false use_fake_hardware:=^|false fake_sensor_commands:=^|false">
-    <xacro:property name="initial_positions" value="${load_yaml(initial_positions_file)['initial_positions']}"/>
-    <ros2_control name="follower" type="system">
-      <xacro:if value="$(arg use_sim)">
-        <hardware>
-          <plugin>gz_ros2_control/GazeboSimSystem</plugin>
-        </hardware>
-      </xacro:if>
-      <xacro:unless value="$(arg use_sim)">
-        <hardware>
-          <xacro:if value="${use_fake_hardware}">
-            <plugin>fake_components/GenericSystem</plugin>
-            <param name="fake_sensor_commands">${fake_sensor_commands}</param>
-            <param name="state_following_offset">0.0</param>
-          </xacro:if>
-          <xacro:unless value="${use_fake_hardware}">
-            <plugin>dynamixel_hardware_interface/DynamixelHardware</plugin>
-            <param name="port_name">/dev/follower</param>
-            <param name="baud_rate">4000000</param>
-            <param name="error_timeout_sec">0.2</param>
-            <param name="dynamixel_model_folder">/param/dxl_model</param>
-            <param name="number_of_joints">19</param>
-            <param name="number_of_transmissions">19</param>
-            <param name="transmission_to_joint_matrix">
-              1, 0, 0, 0, 0, 0, 0, 0, 0, 0, 0, 0, 0, 0, 0, 0, 0, 0, 0,
-              0, 1, 0, 0, 0, 0, 0, 0, 0, 0, 0, 0, 0, 0, 0, 0, 0, 0, 0,
-              0, 0, 1, 0, 0, 0, 0, 0, 0, 0, 0, 0, 0, 0, 0, 0, 0, 0, 0,
-              0, 0, 0, 1, 0, 0, 0, 0, 0, 0, 0, 0, 0, 0, 0, 0, 0, 0, 0,
-              0, 0, 0, 0, 1, 0, 0, 0, 0, 0, 0, 0, 0, 0, 0, 0, 0, 0, 0,
-              0, 0, 0, 0, 0, 1, 0, 0, 0, 0, 0, 0, 0, 0, 0, 0, 0, 0, 0,
-              0, 0, 0, 0, 0, 0, 1, 0, 0, 0, 0, 0, 0, 0, 0, 0, 0, 0, 0,
-              0, 0, 0, 0, 0, 0, 0, 1, 0, 0, 0, 0, 0, 0, 0, 0, 0, 0, 0,
-              0, 0, 0, 0, 0, 0, 0, 0, 1, 0, 0, 0, 0, 0, 0, 0, 0, 0, 0,
-              0, 0, 0, 0, 0, 0, 0, 0, 0, 1, 0, 0, 0, 0, 0, 0, 0, 0, 0,
-              0, 0, 0, 0, 0, 0, 0, 0, 0, 0, 1, 0, 0, 0, 0, 0, 0, 0, 0,
-              0, 0, 0, 0, 0, 0, 0, 0, 0, 0, 0, 1, 0, 0, 0, 0, 0, 0, 0,
-              0, 0, 0, 0, 0, 0, 0, 0, 0, 0, 0, 0, 1, 0, 0, 0, 0, 0, 0,
-              0, 0, 0, 0, 0, 0, 0, 0, 0, 0, 0, 0, 0, 1, 0, 0, 0, 0, 0,
-              0, 0, 0, 0, 0, 0, 0, 0, 0, 0, 0, 0, 0, 0, 1, 0, 0, 0, 0,
-              0, 0, 0, 0, 0, 0, 0, 0, 0, 0, 0, 0, 0, 0, 0, 1, 0, 0, 0,
-              0, 0, 0, 0, 0, 0, 0, 0, 0, 0, 0, 0, 0, 0, 0, 0, 1, 0, 0,
-              0, 0, 0, 0, 0, 0, 0, 0, 0, 0, 0, 0, 0, 0, 0, 0, 0, 1, 0,
-              0, 0, 0, 0, 0, 0, 0, 0, 0, 0, 0, 0, 0, 0, 0, 0, 0, 0, 1
-            </param>
-            <param name="joint_to_transmission_matrix">
-              1, 0, 0, 0, 0, 0, 0, 0, 0, 0, 0, 0, 0, 0, 0, 0, 0, 0, 0,
-              0, 1, 0, 0, 0, 0, 0, 0, 0, 0, 0, 0, 0, 0, 0, 0, 0, 0, 0,
-              0, 0, 1, 0, 0, 0, 0, 0, 0, 0, 0, 0, 0, 0, 0, 0, 0, 0, 0,
-              0, 0, 0, 1, 0, 0, 0, 0, 0, 0, 0, 0, 0, 0, 0, 0, 0, 0, 0,
-              0, 0, 0, 0, 1, 0, 0, 0, 0, 0, 0, 0, 0, 0, 0, 0, 0, 0, 0,
-              0, 0, 0, 0, 0, 1, 0, 0, 0, 0, 0, 0, 0, 0, 0, 0, 0, 0, 0,
-              0, 0, 0, 0, 0, 0, 1, 0, 0, 0, 0, 0, 0, 0, 0, 0, 0, 0, 0,
-              0, 0, 0, 0, 0, 0, 0, 1, 0, 0, 0, 0, 0, 0, 0, 0, 0, 0, 0,
-              0, 0, 0, 0, 0, 0, 0, 0, 1, 0, 0, 0, 0, 0, 0, 0, 0, 0, 0,
-              0, 0, 0, 0, 0, 0, 0, 0, 0, 1, 0, 0, 0, 0, 0, 0, 0, 0, 0,
-              0, 0, 0, 0, 0, 0, 0, 0, 0, 0, 1, 0, 0, 0, 0, 0, 0, 0, 0,
-              0, 0, 0, 0, 0, 0, 0, 0, 0, 0, 0, 1, 0, 0, 0, 0, 0, 0, 0,
-              0, 0, 0, 0, 0, 0, 0, 0, 0, 0, 0, 0, 1, 0, 0, 0, 0, 0, 0,
-              0, 0, 0, 0, 0, 0, 0, 0, 0, 0, 0, 0, 0, 1, 0, 0, 0, 0, 0,
-              0, 0, 0, 0, 0, 0, 0, 0, 0, 0, 0, 0, 0, 0, 1, 0, 0, 0, 0,
-              0, 0, 0, 0, 0, 0, 0, 0, 0, 0, 0, 0, 0, 0, 0, 1, 0, 0, 0,
-              0, 0, 0, 0, 0, 0, 0, 0, 0, 0, 0, 0, 0, 0, 0, 0, 1, 0, 0,
-              0, 0, 0, 0, 0, 0, 0, 0, 0, 0, 0, 0, 0, 0, 0, 0, 0, 1, 0,
-              0, 0, 0, 0, 0, 0, 0, 0, 0, 0, 0, 0, 0, 0, 0, 0, 0, 0, 1
-            </param>
-            <param name="dynamixel_state_pub_msg_name">dynamixel_hardware_interface/dxl_state</param>
-            <param name="get_dynamixel_data_srv_name">dynamixel_hardware_interface/get_dxl_data</param>
-            <param name="set_dynamixel_data_srv_name">dynamixel_hardware_interface/set_dxl_data</param>
-            <param name="reboot_dxl_srv_name">dynamixel_hardware_interface/reboot_dxl</param>
-            <param name="set_dxl_torque_srv_name">dynamixel_hardware_interface/set_dxl_torque</param>
-            <!-- TODO:modification -->
-            <!-- <param name="use_revolute_to_prismatic_gripper">1</param>
-            <param name="revolute_to_prismatic_dxl">dxl81</param>
-            <param name="revolute_max">-1.52</param>
-            <param name="revolute_min">0.92</param>
-            <param name="revolute_to_prismatic_joint">linear_joint</param>
-            <param name="prismatic_max">0.2</param>
-            <param name="prismatic_min">0.0</param> -->
-          </xacro:unless>
-        </hardware>
-      </xacro:unless>
-      <joint name="arm_r_joint1">
-          <command_interface name="position"/>
-          <state_interface name="position">
-          </state_interface>
-          <state_interface name="velocity"/>
-      </joint>
-      <joint name="arm_r_joint2">
-          <command_interface name="position"/>
-          <state_interface name="position">
-          </state_interface>
-          <state_interface name="velocity"/>
-      </joint>
-      <joint name="arm_r_joint3">
-          <command_interface name="position"/>
-          <state_interface name="position">
-          </state_interface>
-          <state_interface name="velocity"/>
-      </joint>
-      <joint name="arm_r_joint4">
-          <command_interface name="position"/>
-          <state_interface name="position">
-          </state_interface>
-          <state_interface name="velocity"/>
-      </joint>
-      <joint name="arm_r_joint5">
-          <command_interface name="position"/>
-          <state_interface name="position">
-          </state_interface>
-          <state_interface name="velocity"/>
-      </joint>
-      <joint name="arm_r_joint6">
-          <command_interface name="position"/>
-          <state_interface name="position">
-          </state_interface>
-          <state_interface name="velocity"/>
-      </joint>
-      <joint name="arm_r_joint7">
-          <command_interface name="position"/>
-          <state_interface name="position">
-          </state_interface>
-          <state_interface name="velocity"/>
-      </joint>
-      <joint name="r_rh_r1_joint">
-        <command_interface name="position"/>
-        <state_interface name="position"/>
-        <state_interface name="velocity"/>
-        <state_interface name="effort"/>
-        <state_interface name="torque_enable"/>
-        <state_interface name="hardware_state"/>
-      </joint>
-      <joint name="arm_l_joint1">
-          <command_interface name="position"/>
-          <state_interface name="position">
-          </state_interface>
-          <state_interface name="velocity"/>
-      </joint>
-      <joint name="arm_l_joint2">
-          <command_interface name="position"/>
-          <state_interface name="position">
-          </state_interface>
-          <state_interface name="velocity"/>
-      </joint>
-      <joint name="arm_l_joint3">
-          <command_interface name="position"/>
-          <state_interface name="position">
-          </state_interface>
-          <state_interface name="velocity"/>
-      </joint>
-      <joint name="arm_l_joint4">
-          <command_interface name="position"/>
-          <state_interface name="position">
-          </state_interface>
-          <state_interface name="velocity"/>
-      </joint>
-      <joint name="arm_l_joint5">
-          <command_interface name="position"/>
-          <state_interface name="position">
-          </state_interface>
-          <state_interface name="velocity"/>
-      </joint>
-      <joint name="arm_l_joint6">
-          <command_interface name="position"/>
-          <state_interface name="position">
-          </state_interface>
-          <state_interface name="velocity"/>
-      </joint>
-      <joint name="arm_l_joint7">
-          <command_interface name="position"/>
-          <state_interface name="position">
-          </state_interface>
-          <state_interface name="velocity"/>
-      </joint>
-      <joint name="l_rh_r1_joint">
-        <command_interface name="position"/>
-        <state_interface name="position"/>
-        <state_interface name="velocity"/>
-        <state_interface name="effort"/>
-        <state_interface name="torque_enable"/>
-        <state_interface name="hardware_state"/>
-      </joint>
-      <joint name="neck_joint1">
-          <command_interface name="position"/>
-          <state_interface name="position">
-          </state_interface>
-          <state_interface name="velocity"/>
-      </joint>
-      <joint name="neck_joint2">
-          <command_interface name="position"/>
-          <state_interface name="position">
-          </state_interface>
-          <state_interface name="velocity"/>
-      </joint>
-      <joint name="linear_joint">
-          <command_interface name="position"/>
-          <state_interface name="position">
-          </state_interface>
-          <state_interface name="velocity"/>
-      </joint>
-      <!-- RIGHT ARM -->
-      <gpio name="dxl1">
-        <param name="type">dxl</param>
-        <param name="ID">1</param>
-        <command_interface name="Goal Position"/>
-        <state_interface name="Present Position"/>
-        <state_interface name="Present Velocity"/>
-        <state_interface name="Torque Enable"/>
-        <state_interface name="Present Input Voltage"/>
-        <param name="Drive Mode">1</param>
-        <param name="Operating Mode">3</param>
-        <param name="Return Delay Time">0</param>
-        <param name="Velocity Limit">2020</param>
-        <param name="Acceleration Limit">20200</param>
-        <param name="Profile Velocity">804</param>
-        <param name="Profile Acceleration">40</param>
-        <param name="Max Position Limit">131072</param>
-        <param name="Min Position Limit">-131072</param>
-        <param name="Position P Gain">1583185</param>
-        <param name="Velocity P Gain">41387</param>
-        <param name="Velocity I Gain">1065630</param>
-      </gpio>
-      <gpio name="dxl2">
-        <param name="type">dxl</param>
-        <param name="ID">2</param>
-        <command_interface name="Goal Position"/>
-        <state_interface name="Present Position"/>
-        <state_interface name="Present Velocity"/>
-        <state_interface name="Torque Enable"/>
-        <state_interface name="Present Input Voltage"/>
-        <param name="Drive Mode">1</param>
-        <param name="Operating Mode">3</param>
-        <param name="Return Delay Time">0</param>
-        <param name="Velocity Limit">2020</param>
-        <param name="Acceleration Limit">20200</param>
-        <param name="Profile Velocity">804</param>
-        <param name="Profile Acceleration">40</param>
-        <param name="Max Position Limit">131072</param>
-        <param name="Min Position Limit">0</param>
-        <param name="Position P Gain">1583185</param>
-        <param name="Velocity P Gain">41387</param>
-        <param name="Velocity I Gain">1065630</param>
-      </gpio>
-      <gpio name="dxl3">
-        <param name="type">dxl</param>
-        <param name="ID">3</param>
-        <command_interface name="Goal Position"/>
-        <state_interface name="Present Position"/>
-        <state_interface name="Present Velocity"/>
-        <state_interface name="Torque Enable"/>
-        <state_interface name="Present Input Voltage"/>
-        <param name="Drive Mode">0</param>
-        <param name="Operating Mode">3</param>
-        <param name="Return Delay Time">0</param>
-        <param name="Velocity Limit">2020</param>
-        <param name="Acceleration Limit">20200</param>
-        <param name="Profile Velocity">804</param>
-        <param name="Profile Acceleration">40</param>
-        <param name="Max Position Limit">262144</param>
-        <param name="Min Position Limit">-262144</param>
-        <param name="Position P Gain">1583185</param>
-        <param name="Velocity P Gain">41387</param>
-        <param name="Velocity I Gain">1065630</param>
-      </gpio>
-      <gpio name="dxl4">
-        <param name="type">dxl</param>
-        <param name="ID">4</param>
-        <command_interface name="Goal Position"/>
-        <state_interface name="Present Position"/>
-        <state_interface name="Present Velocity"/>
-        <state_interface name="Torque Enable"/>
-        <state_interface name="Present Input Voltage"/>
-        <param name="Drive Mode">1</param>
-        <param name="Operating Mode">3</param>
-        <param name="Return Delay Time">0</param>
-        <param name="Velocity Limit">2020</param>
-        <param name="Acceleration Limit">20200</param>
-        <param name="Profile Velocity">804</param>
-        <param name="Profile Acceleration">40</param>
-        <param name="Max Position Limit">160199</param>
-        <param name="Min Position Limit">-160199</param>
-        <param name="Position P Gain">1583185</param>
-        <param name="Velocity P Gain">18184</param>
-        <param name="Velocity I Gain">1085331</param>
-      </gpio>
-      <gpio name="dxl5">
-        <param name="type">dxl</param>
-        <param name="ID">5</param>
-        <command_interface name="Goal Position"/>
-        <state_interface name="Present Position"/>
-        <state_interface name="Present Velocity"/>
-        <state_interface name="Torque Enable"/>
-        <state_interface name="Present Input Voltage"/>
-        <param name="Drive Mode">0</param>
-        <param name="Operating Mode">3</param>
-        <param name="Return Delay Time">0</param>
-        <param name="Velocity Limit">2020</param>
-        <param name="Acceleration Limit">20200</param>
-        <param name="Profile Velocity">804</param>
-        <param name="Profile Acceleration">40</param>
-        <param name="Max Position Limit">262144</param>
-        <param name="Min Position Limit">-262144</param>
-        <param name="Position P Gain">1583185</param>
-        <param name="Velocity P Gain">18184</param>
-        <param name="Velocity I Gain">1085331</param>
-      </gpio>
-      <gpio name="dxl6">
-        <param name="type">dxl</param>
-        <param name="ID">6</param>
-        <command_interface name="Goal Position"/>
-        <state_interface name="Present Position"/>
-        <state_interface name="Present Velocity"/>
-        <state_interface name="Torque Enable"/>
-        <state_interface name="Present Input Voltage"/>
-        <param name="Drive Mode">1</param>
-        <param name="Operating Mode">3</param>
-        <param name="Return Delay Time">0</param>
-        <param name="Velocity Limit">2020</param>
-        <param name="Acceleration Limit">20200</param>
-        <param name="Profile Velocity">804</param>
-        <param name="Profile Acceleration">40</param>
-        <param name="Max Position Limit">131072</param>
-        <param name="Min Position Limit">-131072</param>
-        <param name="Position P Gain">1583185</param>
-        <param name="Velocity P Gain">18184</param>
-        <param name="Velocity I Gain">1085331</param>
-      </gpio>
-      <gpio name="dxl7">
-        <param name="type">dxl</param>
-        <param name="ID">7</param>
-        <command_interface name="Goal Position"/>
-        <state_interface name="Present Position"/>
-        <state_interface name="Present Velocity"/>
-        <state_interface name="Torque Enable"/>
-        <state_interface name="Present Input Voltage"/>
-        <param name="Drive Mode">1</param>
-        <param name="Operating Mode">3</param>
-        <param name="Return Delay Time">0</param>
-        <param name="Profile Velocity">804</param>
-        <param name="Profile Acceleration">40</param>
-        <param name="Max Position Limit">101249</param>
-        <param name="Min Position Limit">-101249</param>
-      </gpio>
-      <gpio name="dxl8">
-        <param name="type">dxl</param>
-        <param name="ID">8</param>
-        <command_interface name="Goal Position"/>
-        <state_interface name="Present Position"/>
-        <state_interface name="Present Velocity"/>
-        <state_interface name="Present Current"/>
-        <state_interface name="Torque Enable"/>
-        <state_interface name="Present Input Voltage"/>
-        <param name="Operating Mode">5</param>
-        <param name="Return Delay Time">0</param>
-      </gpio>
-      <!-- LEFT ARM -->
-      <gpio name="dxl31">
-        <param name="type">dxl</param>
-        <param name="ID">31</param>
-        <command_interface name="Goal Position"/>
-        <state_interface name="Present Position"/>
-        <state_interface name="Present Velocity"/>
-        <state_interface name="Torque Enable"/>
-        <state_interface name="Present Input Voltage"/>
-        <param name="Drive Mode">0</param>
-        <param name="Operating Mode">3</param>
-        <param name="Return Delay Time">0</param>
-        <param name="Velocity Limit">2020</param>
-        <param name="Acceleration Limit">20200</param>
-        <param name="Profile Velocity">804</param>
-        <param name="Profile Acceleration">40</param>
-        <param name="Max Position Limit">131072</param>
-        <param name="Min Position Limit">-131072</param>
-        <param name="Position P Gain">1583185</param>
-        <param name="Velocity P Gain">41387</param>
-        <param name="Velocity I Gain">1065630</param>
-      </gpio>
-      <gpio name="dxl32">
-        <param name="type">dxl</param>
-        <param name="ID">32</param>
-        <command_interface name="Goal Position"/>
-        <state_interface name="Present Position"/>
-        <state_interface name="Present Velocity"/>
-        <state_interface name="Torque Enable"/>
-        <state_interface name="Present Input Voltage"/>
-        <param name="Drive Mode">0</param>
-        <param name="Operating Mode">3</param>
-        <param name="Return Delay Time">0</param>
-        <param name="Velocity Limit">2020</param>
-        <param name="Acceleration Limit">20200</param>
-        <param name="Profile Velocity">804</param>
-        <param name="Profile Acceleration">40</param>
-        <param name="Max Position Limit">131072</param>
-        <param name="Min Position Limit">0</param>
-        <param name="Position P Gain">1583185</param>
-        <param name="Velocity P Gain">41387</param>
-        <param name="Velocity I Gain">1065630</param>
-      </gpio>
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