Commit message: Update follower URDF and STL files: Modify joint origins for arm links, add D405 camera sensors.

File: ffw_description/urdf/follower/ffw_follower_body.urdf.xacro (robot description, xacro)
@@ -1,4 +1,5 @@
 <?xml version="1.0" encoding="UTF-8"?>
 <robot xmlns:xacro="http://www.ros.org/wiki/xacro" name="ffw">
+   <xacro:include filename="$(find realsense2_description)/urdf/_d405.urdf.xacro" />
    <xacro:property name="meshes_file_direction" value="package://ffw_description/meshes/follower" />
    <link name="base_link">
@@ -297,5 +298,5 @@
       <parent link="arm_r_link6" />
       <child link="arm_r_link7" />
-      <origin xyz="0 0 0" rpy="0 0 0" />
+      <origin xyz="0 -0.0006 0" rpy="0 0 0" />
       <axis xyz="1 0 0" />
       <limit velocity="4.8" effort="1000" lower="-0.3" upper="1.57" />
@@ -324,4 +325,7 @@
       </inertial>
    </link>
+   <xacro:sensor_d405 parent="arm_r_link7" use_nominal_extrinsics="false" name="camera_r">
+      <origin xyz="0.102293 -0.021 -0.0345518" rpy="-1.57079632679 1.66678943569 0"/>
+   </xacro:sensor_d405>
    <joint name="arm_l_joint1" type="revolute">
       <parent link="arm_base_link" />
@@ -507,5 +511,5 @@
       <parent link="arm_l_link6" />
       <child link="arm_l_link7" />
-      <origin xyz="0 0 0" rpy="0 0 0" />
+      <origin xyz="0 0.0006 0" rpy="0 0 0" />
       <axis xyz="1 0 0" />
       <limit velocity="4.8" effort="1000" lower="-1.57" upper="0.3" />
@@ -534,3 +538,6 @@
       </inertial>
    </link>
+   <xacro:sensor_d405 parent="arm_l_link7" use_nominal_extrinsics="false" name="camera_l">
+      <origin xyz="0.102293 -0.021 -0.0345518" rpy="-1.57079632679 1.66678943569 0"/>
+   </xacro:sensor_d405>
 </robot>

File: ffw_description/urdf/follower/ffw_follower_with_rh.urdf.xacro (robot description, xacro)
@@ -21,5 +21,5 @@
   </joint>
   <joint name="left_hand_fixed" type="fixed">
-    <origin xyz="0 0 -0.05" rpy="0 3.14 -1.57"/>
+    <origin xyz="0 0 -0.05" rpy="0 3.14159265359 0"/>
     <parent link="arm_l_link7"/>
     <axis xyz="0 0 0"/>
@@ -27,5 +27,5 @@
   </joint>
   <joint name="right_hand_fixed" type="fixed">
-    <origin xyz="0 0 -0.05" rpy="0 3.14 1.57"/>
+    <origin xyz="0 0 -0.05" rpy="0 3.14159265359 0"/>
     <parent link="arm_r_link7"/>
     <axis xyz="0 0 0"/>
