Commit message: Refactor URDF file to update joint and link names for consistency, and adjust sensor command references for improved integration.

File: ffw_description/urdf/ffw_lg2_leader/ffw_lg2_leader.urdf.xacro (robot description, xacro)
@@ -5,25 +5,27 @@
   <xacro:arg name="fake_sensor_commands" default="false" />
   <xacro:arg name="prefix" default="" />
-  <xacro:include filename="$(find ffw_description)/urdf/leader/ffw_leader_body.urdf.xacro" />
-  <xacro:include filename="$(find ffw_description)/ros2_control/ffw_lg2_leader/ffw_lg2_leader_left_system.ros2_control.xacro" />
-  <xacro:include filename="$(find ffw_description)/ros2_control/ffw_lg2_leader/ffw_lg2_leader_right_system.ros2_control.xacro" />
+  <xacro:include filename="$(find ffw_description)/urdf/common/leader/ffw_leader_body.urdf.xacro" />
+  <xacro:include filename="$(find ffw_description)/ros2_control/ffw_lg2_leader/ffw_lg2_leader_left.ros2_control.xacro" />
+  <xacro:include filename="$(find ffw_description)/ros2_control/ffw_lg2_leader/ffw_lg2_leader_right.ros2_control.xacro" />
   <link name="world"/>
-  <xacro:ffw_leader_body parent="world" prefix="${prefix}">
+  <xacro:ffw_leader_body parent="$(arg prefix)world" prefix="$(arg prefix)">
     <origin xyz="0 0 0" rpy="0 0 0" />
   </xacro:ffw_leader_body>
-  <joint name="${prefix}gripper_l_joint" type="revolute">
+  <joint name="$(arg prefix)gripper_l_joint1" type="revolute">
     <origin xyz="0 0 0" rpy="0 0 0"/>
-    <parent link="${prefix}arm_l_link7"/>
+    <parent link="$(arg prefix)arm_l_link7"/>
     <axis xyz="0 1 0"/>
-    <child link="${prefix}gripper_l_link"/>
+    <child link="$(arg prefix)gripper_l_link1"/>
+    <limit velocity="6.5" effort="1000" lower="-6.28" upper="6.28" />
   </joint>
-  <link name="${prefix}gripper_l_link"/>
-  <joint name="${prefix}gripper_r_joint" type="revolute">
+  <link name="$(arg prefix)gripper_l_link1"/>
+  <joint name="$(arg prefix)gripper_r_joint1" type="revolute">
     <origin xyz="0 0 0" rpy="0 0 0"/>
-    <parent link="${prefix}arm_r_link7"/>
+    <parent link="$(arg prefix)arm_r_link7"/>
     <axis xyz="0 1 0"/>
-    <child link="${prefix}gripper_r_link"/>
+    <child link="$(arg prefix)gripper_r_link1"/>
+    <limit velocity="6.5" effort="1000" lower="-6.28" upper="6.28" />
   </joint>
-  <link name="${prefix}gripper_r_link"/>
+  <link name="$(arg prefix)gripper_r_link1"/>
   <xacro:ffw_lg2_leader_left_system
       use_sim="$(arg use_sim)"
