Commit message: Modified files for gazebo
Signed-off-by: Wonho Yun <ywh@robotis.com>

File: ffw_description/urdf/common/rh_p12_rn_a/rh_p12_rn_a.urdf.xacro (robot description, xacro)
@@ -74,5 +74,5 @@
       <limit velocity="6.5" effort="1000" lower="0.0" upper="1.0" />
       <dynamics damping="0.7"/>
-      <mimic joint="${prefix}rh_r1_joint" multiplier="1"/>
+      <mimic joint="${prefix}joint1" multiplier="1"/>
     </joint>
     <!-- rh_p12_rn_r2 -->
@@ -107,5 +107,5 @@
       <limit velocity="6.5" effort="1000" lower="0.0" upper="1.1" />
       <dynamics damping="0.7"/>
-      <mimic joint="${prefix}rh_r1_joint" multiplier="1"/>
+      <mimic joint="${prefix}joint1" multiplier="1"/>
     </joint>
     <!-- rh_p12_rn_l1 -->
@@ -140,5 +140,5 @@
       <limit velocity="6.5" effort="1000" lower="0.0" upper="1.0" />
       <dynamics damping="0.7"/>
-      <mimic joint="${prefix}rh_r1_joint" multiplier="1"/>
+      <mimic joint="${prefix}joint1" multiplier="1"/>
     </joint>
     <!-- rh_p12_rn_l2 -->

File: ffw_description/urdf/ffw_bg2_follower/ffw_bg2_follower.urdf.xacro (robot description, xacro)
@@ -53,5 +53,5 @@
   <gazebo>
       <plugin filename="gz_ros2_control-system" name="gz_ros2_control::GazeboSimROS2ControlPlugin">
-        <parameters>$(find ffw_bringup)/config/ffw_bg2_follower_gazebo_controller_manager.yaml</parameters>
+        <parameters>$(find ffw_bringup)/config/ffw_bg2_follower/ffw_bg2_follower_gazebo_controller_manager.yaml</parameters>
       </plugin>
   </gazebo>
