Commit message: Updated STL files for follower model and added new meshes for revision  4, including arm links and body assembly. Adjusted URDF and XACRO files for improved joint configurations and limits in the ffw_bg2_rev4_follower setup.

File: ffw_description/ros2_control/ffw_bg2_rev4_follower/ffw_bg2_follower.ros2_control.xacro (robot description, xacro)
@@ -202,5 +202,5 @@
         <param name="Profile Acceleration">300</param>
         <param name="Max Position Limit">0</param>
-        <param name="Min Position Limit">-131072</param>
+        <param name="Min Position Limit">-262144</param>
         <param name="Position P Gain">1583185</param>
         <param name="Velocity P Gain">41387</param>
@@ -239,5 +239,5 @@
         <param name="Profile Velocity">2020</param>
         <param name="Profile Acceleration">300</param>
-        <param name="Max Position Limit">160199</param>
+        <param name="Max Position Limit">90000</param>
         <param name="Min Position Limit">-245000</param>
         <param name="Position P Gain">1583185</param>
@@ -342,5 +342,5 @@
         <param name="Profile Velocity">2020</param>
         <param name="Profile Acceleration">300</param>
-        <param name="Max Position Limit">131072</param>
+        <param name="Max Position Limit">262144</param>
         <param name="Min Position Limit">0</param>
         <param name="Position P Gain">1583185</param>
@@ -380,5 +380,5 @@
         <param name="Profile Velocity">2020</param>
         <param name="Profile Acceleration">300</param>
-        <param name="Max Position Limit">160199</param>
+        <param name="Max Position Limit">90000</param>
         <param name="Min Position Limit">-245000</param>
         <param name="Position P Gain">1583185</param>
@@ -482,5 +482,5 @@
         <param name="Profile Velocity">200</param>
         <param name="Profile Acceleration">50</param>
-        <param name="Max Position Limit">2731</param>
+        <param name="Max Position Limit">2500</param>
         <param name="Min Position Limit">1896</param>
         <param name="Position P Gain">1600</param>

File: ffw_description/urdf/ffw_bg2_rev3_follower/ffw_follower_body.xacro (robot description, xacro)
@@ -3,5 +3,5 @@
    <xacro:macro name="ffw_follower_body" params="prefix parent *origin">
       <xacro:include filename="$(find realsense2_description)/urdf/_d405.urdf.xacro" />
-      <xacro:property name="meshes_file_direction" value="package://ffw_description/meshes/common/follower" />
+      <xacro:property name="meshes_file_direction" value="package://ffw_description/meshes/ffw_bg2_rev3_follower" />
       <joint name="${prefix}lift_joint" type="prismatic">
          <parent link="${parent}"/>
@@ -37,7 +37,7 @@
          <parent link="${prefix}arm_base_link" />
          <child link="${prefix}head_link1" />
-         <origin xyz="0.0494878 0 0.102123" rpy="0 0 0" />
-         <axis xyz="0 1 0" />
-         <limit velocity="4.8" effort="1000" lower="-0.2317" upper="0.6951" />
+         <origin xyz="0.019 0 0.06475" rpy="0 0 0" />
+         <axis xyz="0 1 0" />
+         <limit velocity="4.8" effort="1000" lower="0.0" upper="0.4" />
          <dynamics damping="0.1" />
       </joint>
@@ -67,7 +67,7 @@
          <parent link="${prefix}head_link1" />
          <child link="${prefix}head_link2" />
-         <origin xyz="0.0365694 0 0.0563797" rpy="0 0 0" />
+         <origin xyz="0 0 0.0475" rpy="0 0 0" />
          <axis xyz="0 0 1" />
-         <limit velocity="4.8" effort="1000" lower="-0.35" upper="0.35" />
+         <limit velocity="4.8" effort="1000" lower="-0.6" upper="0.6" />
          <dynamics damping="0.1" />
       </joint>
@@ -97,5 +97,5 @@
          <parent link="${prefix}arm_base_link" />
          <child link="${prefix}arm_l_link1" />
-         <origin xyz="0 0.1045 0" rpy="0 0 0" />
+         <origin xyz="0 0.11345 0" rpy="0 0 0" />
          <axis xyz="0 1 0" />
          <limit velocity="4.8" effort="1000" lower="-3.14" upper="3.14" />
@@ -127,5 +127,5 @@
          <parent link="${prefix}arm_l_link1" />
          <child link="${prefix}arm_l_link2" />
-         <origin xyz="0 0.123 0" rpy="0 0 0" />
+         <origin xyz="0 0.11205 0" rpy="0 0 0" />
          <axis xyz="1 0 0" />
          <limit velocity="4.8" effort="1000" lower="0.0" upper="3.14" />
@@ -157,5 +157,5 @@
          <parent link="${prefix}arm_l_link2" />
          <child link="${prefix}arm_l_link3" />
-         <origin xyz="0 0 -0.165" rpy="0 0 0" />
+         <origin xyz="0 0 -0.17595" rpy="0 0 0" />
          <axis xyz="0 0 1" />
          <limit velocity="4.8" effort="1000" lower="-3.14" upper="3.14" />
@@ -187,7 +187,7 @@
          <parent link="${prefix}arm_l_link3" />
          <child link="${prefix}arm_l_link4" />
-         <origin xyz="0.041004 0 -0.135" rpy="0 0 0" />
-         <axis xyz="0 1 0" />
-         <limit velocity="4.8" effort="1000" lower="-2.9361" upper="1.0786" />
+         <origin xyz="0 0 -0.10605" rpy="0 0 0" />
+         <axis xyz="0 1 0" />
+         <limit velocity="4.8" effort="1000" lower="-1.86" upper="1.86" />
          <dynamics damping="0.1" />
       </joint>
@@ -217,5 +217,5 @@
          <parent link="${prefix}arm_l_link4" />
          <child link="${prefix}arm_l_link5" />
-         <origin xyz="-0.041004 0 -0.1489" rpy="0 0 0" />
+         <origin xyz="0 0 -0.16595" rpy="0 0 0" />
          <axis xyz="0 0 1" />
          <limit velocity="4.8" effort="1000" lower="-3.14" upper="3.14" />
@@ -247,7 +247,7 @@
          <parent link="${prefix}arm_l_link5" />
          <child link="${prefix}arm_l_link6" />
-         <origin xyz="0 0 -0.1041" rpy="0 0 0" />
-         <axis xyz="0 1 0" />
-         <limit velocity="4.8" effort="1000" lower="-1.57" upper="1.57" />
+         <origin xyz="0 0 -0.1593" rpy="0 0 0" />
+         <axis xyz="0 1 0" />
+         <limit velocity="4.8" effort="1000" lower="-0.5" upper="0.5" />
          <dynamics damping="0.1" />
       </joint>
@@ -277,7 +277,7 @@
          <parent link="${prefix}arm_l_link6" />
          <child link="${prefix}arm_l_link7" />
-         <origin xyz="0 0 -0.0885" rpy="0 0 0" />
+         <origin xyz="0 0.0006 0" rpy="0 0 0" />
          <axis xyz="1 0 0" />
-         <limit velocity="4.8" effort="1000" lower="-1.8201" upper="1.5804" />
+         <limit velocity="4.8" effort="1000" lower="-1.57" upper="0.3" />
          <dynamics damping="0.1" />
       </joint>
@@ -305,10 +305,10 @@
       </link>
       <xacro:sensor_d405 parent="${prefix}arm_l_link7" use_nominal_extrinsics="false" name="${prefix}camera_l">
-         <origin xyz="0.108236 -0.021 -0.062552" rpy="-1.57079632679 1.66678943569 0"/>
+         <origin xyz="0.102293 -0.021 -0.0345518" rpy="-1.57079632679 1.66678943569 0"/>
       </xacro:sensor_d405>
       <joint name="${prefix}arm_r_joint1" type="revolute">
          <parent link="${prefix}arm_base_link" />
          <child link="${prefix}arm_r_link1" />
-         <origin xyz="0 -0.1045 0" rpy="0 0 0" />
+         <origin xyz="0 -0.11345 0" rpy="0 0 0" />
          <axis xyz="0 1 0" />
          <limit velocity="4.8" effort="1000" lower="-3.14" upper="3.14" />
@@ -340,5 +340,5 @@
          <parent link="${prefix}arm_r_link1" />
          <child link="${prefix}arm_r_link2" />
-         <origin xyz="0 -0.123 0" rpy="0 0 0" />
+         <origin xyz="0 -0.11205 0" rpy="0 0 0" />
          <axis xyz="1 0 0" />
          <limit velocity="4.8" effort="1000" lower="-3.14" upper="0" />
@@ -370,5 +370,5 @@
          <parent link="${prefix}arm_r_link2" />
          <child link="${prefix}arm_r_link3" />
-         <origin xyz="0 0 -0.165" rpy="0 0 0" />
+         <origin xyz="0 0 -0.175950" rpy="0 0 0" />
          <axis xyz="0 0 1" />
          <limit velocity="4.8" effort="1000" lower="-3.14" upper="3.14" />
@@ -400,7 +400,7 @@
          <parent link="${prefix}arm_r_link3" />
          <child link="${prefix}arm_r_link4" />
-         <origin xyz="0.041004 0 -0.135" rpy="0 0 0" />
-         <axis xyz="0 1 0" />
-         <limit velocity="4.8" effort="1000" lower="-2.9361" upper="1.0786" />
+         <origin xyz="0 0 -0.10605" rpy="0 0 0" />
+         <axis xyz="0 1 0" />
+         <limit velocity="4.8" effort="1000" lower="-1.86" upper="1.86" />
          <dynamics damping="0.1" />
       </joint>
@@ -430,5 +430,5 @@
          <parent link="${prefix}arm_r_link4" />
          <child link="${prefix}arm_r_link5" />
-         <origin xyz="-0.041004 0 -0.1489" rpy="0 0 0" />
+         <origin xyz="0 0 -0.16595" rpy="0 0 0" />
          <axis xyz="0 0 1" />
          <limit velocity="4.8" effort="1000" lower="-3.14" upper="3.14" />
@@ -460,7 +460,7 @@
          <parent link="${prefix}arm_r_link5" />
          <child link="${prefix}arm_r_link6" />
-         <origin xyz="0 0 -0.1041" rpy="0 0 0" />
-         <axis xyz="0 1 0" />
-         <limit velocity="4.8" effort="1000" lower="-1.57" upper="1.57" />
+         <origin xyz="0 0 -0.1593" rpy="0 0 0" />
+         <axis xyz="0 1 0" />
+         <limit velocity="4.8" effort="1000" lower="-0.6" upper="0.6" />
          <dynamics damping="0.1" />
       </joint>
@@ -490,7 +490,7 @@
          <parent link="${prefix}arm_r_link6" />
          <child link="${prefix}arm_r_link7" />
-         <origin xyz="0 0 -0.0885" rpy="0 0 0" />
+         <origin xyz="0 -0.0006 0" rpy="0 0 0" />
          <axis xyz="1 0 0" />
-         <limit velocity="4.8" effort="1000" lower="-1.5804" upper="1.8201" />
+         <limit velocity="4.8" effort="1000" lower="-0.3" upper="1.57" />
          <dynamics damping="0.1" />
       </joint>
@@ -518,5 +518,5 @@
       </link>
       <xacro:sensor_d405 parent="${prefix}arm_r_link7" use_nominal_extrinsics="false" name="${prefix}camera_r">
-         <origin xyz="0.108236 -0.021 -0.062552" rpy="-1.57079632679 1.66678943569 0"/>
+         <origin xyz="0.102293 -0.021 -0.0345518" rpy="-1.57079632679 1.66678943569 0"/>
       </xacro:sensor_d405>
    </xacro:macro>

File: ffw_description/urdf/ffw_bg2_rev4_follower/ffw_bg2_follower.urdf.xacro (robot description, xacro)
@@ -40,11 +40,11 @@
   </link>
   <xacro:ffw_follower_body parent="$(arg prefix)base_link" prefix="$(arg prefix)">
-    <origin xyz="0.053 0 1.2846" rpy="0 0 0" />
+    <origin xyz="0.0055 0 1.4316" rpy="0 0 0" />
   </xacro:ffw_follower_body>
   <xacro:rh_p12_rn_a parent="$(arg prefix)arm_l_link7" prefix="$(arg prefix)gripper_l_">
-    <origin xyz="0 0 -0.05" rpy="0 3.14159265359 0"/>
+    <origin xyz="0 0 -0.078" rpy="0 3.14159265359 0"/>
   </xacro:rh_p12_rn_a>
   <xacro:rh_p12_rn_a parent="$(arg prefix)arm_r_link7" prefix="$(arg prefix)gripper_r_">
-    <origin xyz="0 0 -0.05" rpy="0 3.14159265359 0"/>
+    <origin xyz="0 0 -0.078" rpy="0 3.14159265359 0"/>
   </xacro:rh_p12_rn_a>
   <xacro:ffw_bg2_follower_system
