Commit message: Update follower configurations and joint limits in URDF and launch files for improved trajectory control and consistency across the system.

File: ffw_description/urdf/common/follower/ffw_follower_body.xacro (robot description, xacro)
@@ -9,5 +9,5 @@
          <xacro:insert_block name="origin" />
          <axis xyz="0 0 1" />
-         <limit velocity="4.8" effort="1000" lower="0.0" upper="0.25" />
+         <limit velocity="4.8" effort="1000" lower="-0.5" upper="0.0" />
          <dynamics damping="0.1" />
       </joint>

Commit message: Updated STL files for follower model, including arm links and body assembly, and removed inertial properties from URDF and XACRO files for the ffw_bg2_rev4_follower setup.

File: ffw_description/urdf/common/follower/ffw_follower_body.xacro (robot description, xacro)
@@ -28,9 +28,4 @@
             </geometry>
          </collision>
-         <inertial>
-            <origin xyz="-4.607316100e-02 -2.281005300e-05 -2.702082100e-02" />
-            <mass value="8.721758400e+00" />
-            <inertia ixx="9.316905600e-02" ixy="1.223827600e-05" ixz="-1.109867300e-02" iyy="5.761433200e-02" iyz="-1.525995300e-05" izz="9.659478800e-02" />
-         </inertial>
       </link>
       <joint name="${prefix}head_joint1" type="revolute">
@@ -58,9 +53,4 @@
             </geometry>
          </collision>
-         <inertial>
-            <origin xyz="-7.329875400e-03 0.000000000e+00 4.343627400e-02" />
-            <mass value="1.394727200e-01" />
-            <inertia ixx="5.752068900e-05" ixy="0.000000000e+00" ixz="4.943420800e-06" iyy="6.544451100e-05" iyz="0.000000000e+00" izz="5.003265300e-05" />
-         </inertial>
       </link>
       <joint name="${prefix}head_joint2" type="revolute">
@@ -88,9 +78,4 @@
             </geometry>
          </collision>
-         <inertial>
-            <origin xyz="8.779073500e-03 -8.403922700e-05 4.254319200e-02" />
-            <mass value="1.450781500e-01" />
-            <inertia ixx="1.834982400e-04" ixy="-4.755711300e-08" ixz="-3.507748300e-06" iyy="2.283875600e-05" iyz="-2.683629200e-08" izz="1.834735800e-04" />
-         </inertial>
       </link>
       <joint name="${prefix}arm_l_joint1" type="revolute">
@@ -118,9 +103,4 @@
             </geometry>
          </collision>
-         <inertial>
-            <origin xyz="1.625390900e-02 1.150971200e-01 1.160152700e-04" />
-            <mass value="1.933953700e+00" />
-            <inertia ixx="2.404898000e-03" ixy="-2.558530200e-04" ixz="1.123409700e-05" iyy="2.562086300e-03" iyz="-2.410406700e-06" izz="3.054703500e-03" />
-         </inertial>
       </link>
       <joint name="${prefix}arm_l_joint2" type="revolute">
@@ -148,9 +128,4 @@
             </geometry>
          </collision>
-         <inertial>
-            <origin xyz="9.096806400e-03 -1.055040600e-04 -1.440332700e-01" />
-            <mass value="2.124140800e+00" />
-            <inertia ixx="9.942940700e-03" ixy="-1.417843000e-06" ixz="-2.368306000e-03" iyy="1.085364600e-02" iyz="4.864401200e-06" izz="3.162675400e-03" />
-         </inertial>
       </link>
       <joint name="${prefix}arm_l_joint3" type="revolute">
@@ -178,9 +153,4 @@
             </geometry>
          </collision>
-         <inertial>
-            <origin xyz="2.510915400e-05 1.794721700e-02 -1.087573700e-01" />
-            <mass value="1.407742700e+00" />
-            <inertia ixx="1.933549600e-03" ixy="1.416541700e-06" ixz="3.403693800e-07" iyy="1.449111500e-03" iyz="2.119230000e-04" izz="1.573054500e-03" />
-         </inertial>
       </link>
       <joint name="${prefix}arm_l_joint4" type="revolute">
@@ -208,9 +178,4 @@
             </geometry>
          </collision>
-         <inertial>
-            <origin xyz="-4.397034900e-05 9.787041900e-03 -1.378883000e-01" />
-            <mass value="1.513136300e+00" />
-            <inertia ixx="6.362873000e-03" ixy="-6.975278900e-07" ixz="1.270290600e-06" iyy="5.687568700e-03" iyz="-1.606244800e-03" izz="1.926579800e-03" />
-         </inertial>
       </link>
       <joint name="${prefix}arm_l_joint5" type="revolute">
@@ -238,9 +203,4 @@
             </geometry>
          </collision>
-         <inertial>
-            <origin xyz="-4.953061500e-05 1.879570900e-02 -9.836393300e-02" />
-            <mass value="1.344193200e+00" />
-            <inertia ixx="1.699126800e-03" ixy="-3.352286000e-06" ixz="-4.262511700e-07" iyy="1.234144700e-03" iyz="1.491721400e-04" izz="1.502606200e-03" />
-         </inertial>
       </link>
       <joint name="${prefix}arm_l_joint6" type="revolute">
@@ -268,9 +228,4 @@
             </geometry>
          </collision>
-         <inertial>
-            <origin xyz="3.844904400e-04 1.942979300e-02 -6.394564400e-02" />
-            <mass value="6.362337700e-01" />
-            <inertia ixx="1.388910800e-03" ixy="4.568060400e-06" ixz="5.660750700e-06" iyy="1.086005700e-03" iyz="-5.260047400e-04" izz="9.664181300e-04" />
-         </inertial>
       </link>
       <joint name="${prefix}arm_l_joint7" type="revolute">
@@ -298,9 +253,4 @@
             </geometry>
          </collision>
-         <inertial>
-            <origin xyz="-7.210928100e-03 0.000000000e+00 -2.560159000e-02" />
-            <mass value="1.243248700e-01" />
-            <inertia ixx="5.994976500e-05" ixy="0.000000000e+00" ixz="2.416233500e-05" iyy="1.738725800e-04" iyz="0.000000000e+00" izz="1.599468200e-04" />
-         </inertial>
       </link>
       <xacro:sensor_d405 parent="${prefix}arm_l_link7" use_nominal_extrinsics="false" name="${prefix}camera_l">
@@ -331,9 +281,4 @@
             </geometry>
          </collision>
-         <inertial>
-            <origin xyz="1.624540100e-02 -1.150833200e-01 -1.160152700e-04" />
-            <mass value="1.933953700e+00" />
-            <inertia ixx="2.404191600e-03" ixy="2.572789100e-04" ixz="-1.117177300e-05" iyy="2.564101300e-03" iyz="-2.413538900e-06" izz="3.056035500e-03" />
-         </inertial>
       </link>
       <joint name="${prefix}arm_r_joint2" type="revolute">
@@ -361,9 +306,4 @@
             </geometry>
          </collision>
-         <inertial>
-            <origin xyz="9.040963900e-03 1.058016600e-04 -1.440332700e-01" />
-            <mass value="2.124140800e+00" />
-            <inertia ixx="9.942940500e-03" ixy="2.652646000e-06" ixz="-2.364645000e-03" iyy="1.085582700e-02" iyz="-4.964042700e-06" izz="3.164856100e-03" />
-         </inertial>
       </link>
       <joint name="${prefix}arm_r_joint3" type="revolute">
@@ -391,9 +331,4 @@
             </geometry>
          </collision>
-         <inertial>
-            <origin xyz="-2.510915300e-05 -1.794721700e-02 -1.087648400e-01" />
-            <mass value="1.407742700e+00" />
-            <inertia ixx="1.932711900e-03" ixy="2.160084900e-06" ixz="-3.401052700e-07" iyy="1.448297100e-03" iyz="-2.117341800e-04" izz="1.573054500e-03" />
-         </inertial>
       </link>
       <joint name="${prefix}arm_r_joint4" type="revolute">
@@ -421,9 +356,4 @@
             </geometry>
          </collision>
-         <inertial>
-            <origin xyz="4.397034900e-05 -9.787357900e-03 -1.378883000e-01" />
-            <mass value="1.513136300e+00" />
-            <inertia ixx="6.362933700e-03" ixy="-6.975489100e-07" ixz="-1.270290600e-06" iyy="5.687568700e-03" iyz="1.606295500e-03" izz="1.926640600e-03" />
-         </inertial>
       </link>
       <joint name="${prefix}arm_r_joint5" type="revolute">
@@ -451,9 +381,4 @@
             </geometry>
          </collision>
-         <inertial>
-            <origin xyz="-2.629623700e-05 -1.879570800e-02 -9.838709700e-02" />
-            <mass value="1.344193200e+00" />
-            <inertia ixx="1.697614400e-03" ixy="1.382419000e-06" ixz="-2.509507400e-07" iyy="1.234418100e-03" iyz="-1.480093000e-04" izz="1.504563200e-03" />
-         </inertial>
       </link>
       <joint name="${prefix}arm_r_joint6" type="revolute">
@@ -481,9 +406,4 @@
             </geometry>
          </collision>
-         <inertial>
-            <origin xyz="3.398392800e-04 -1.943041700e-02 -6.394589600e-02" />
-            <mass value="6.362337700e-01" />
-            <inertia ixx="1.388961300e-03" ixy="-4.201514200e-06" ixz="5.358941000e-06" iyy="1.086005700e-03" iyz="5.260231200e-04" izz="9.664532300e-04" />
-         </inertial>
       </link>
       <joint name="${prefix}arm_r_joint7" type="revolute">
@@ -511,9 +431,4 @@
             </geometry>
          </collision>
-         <inertial>
-            <origin xyz="-7.379093300e-03 0.000000000e+00 -2.559652800e-02" />
-            <mass value="1.243248700e-01" />
-            <inertia ixx="5.998355100e-05" ixy="0.000000000e+00" ixz="2.451378300e-05" iyy="1.746288100e-04" iyz="0.000000000e+00" izz="1.606692600e-04" />
-         </inertial>
       </link>
       <xacro:sensor_d405 parent="${prefix}arm_r_link7" use_nominal_extrinsics="false" name="${prefix}camera_r">

File: ffw_description/urdf/ffw_bg2_rev4_follower/ffw_bg2_follower.urdf.xacro (robot description, xacro)
@@ -33,9 +33,4 @@
         </geometry>
     </collision>
-    <inertial>
-        <origin xyz="-4.215593900e-02 1.414784900e-03 5.544221100e-01" />
-        <mass value="7.208755500e+01" />
-        <inertia ixx="2.239045300e+01" ixy="-1.263524100e-02" ixz="2.036407800e+00" iyy="2.283017500e+01" iyz="3.941520900e-02" izz="2.211418500e+00" />
-    </inertial>
   </link>
   <xacro:ffw_follower_body parent="$(arg prefix)base_link" prefix="$(arg prefix)">
