Commit message: Update URDF file to use package-relative mesh paths for the d405 model, improving portability.

File: ffw_description/urdf/ffw_bg2_rev4_follower/ffw_bg2_follower.urdf (robot description, URDF)
Before this commit: robot ffw_bg2_follower, 33 links, 32 joints
Links:
- link camera_l_link: geometry collision box size=0.023 0.042 0.042; visual mesh filename=package://realsense2_description/meshes/d405.stl scale=0.001 0.001 0.001
- link camera_r_link: geometry collision box size=0.023 0.042 0.042; visual mesh filename=package://realsense2_description/meshes/d405.stl scale=0.001 0.001 0.001
