Commit message: Update joystick calibration values and add swerve drive controller configuration
- Adjusted joystick calibration center and max values in ffw_lg2_leader AI hardware controller configuration.
- Introduced swerve drive controller parameters in ffw_sg2_follower AI hardware controller configuration.
- Updated launch file to include swerve drive controller.
- Enhanced URDF and XACRO files to incorporate swerve drive components and configurations.
- Modified joint trajectory command broadcaster to remove swerve mode check.
- Adjusted joystick controller to scale command velocities for swerve mode.

File: ffw_description/ros2_control/ffw_sg2_rev1_follower/ffw_sg2_follower.ros2_control.xacro (robot description, xacro)
@@ -3,5 +3,5 @@
   <xacro:macro name="ffw_sg2_follower_system" params="use_sim:=^|false use_fake_hardware:=^|false fake_sensor_commands:=^|false">
     <xacro:property name="initial_positions" value="${load_yaml(initial_positions_file)['initial_positions']}"/>
-    <ros2_control name="ffw_sg2_follower" type="system">
+    <ros2_control name="ffw_sg2_follower" type="system" is_async="true">
       <xacro:if value="$(arg use_sim)">
         <hardware>

File: ffw_description/urdf/ffw_sg2_rev1_follower/ffw_sg2_follower.urdf.xacro (robot description, xacro)
@@ -10,4 +10,5 @@
   <xacro:include filename="$(find ffw_description)/urdf/common/rh_p12_rn_a/rh_p12_rn_a.urdf.xacro" />
   <xacro:include filename="$(find ffw_description)/ros2_control/$(arg model)/ffw_sg2_follower.ros2_control.xacro" />
+  <xacro:include filename="$(find ffw_description)/ros2_control/$(arg model)/ffw_sg2_base.ros2_control.xacro" />
   <xacro:include filename="$(find ffw_description)/gazebo/$(arg model)/ffw_sg2_follower.gazebo.xacro" />
   <link name="world"/>
@@ -50,5 +51,57 @@
     <origin xyz="0 0 -0.078" rpy="0 3.14159265359 0"/>
   </xacro:rh_p12_rn_a>
+  <link name="$(arg prefix)link_1"/>
+  <joint name="$(arg prefix)joint1_steer" type="revolute">
+      <parent link="$(arg prefix)base_link"/>
+      <child link="$(arg prefix)link_1"/>
+      <origin xyz="0.2135 0.2554 0" rpy="0 0 0"/>
+      <axis xyz="0 0 1" />
+      <limit velocity="4.8" effort="1" lower="${-pi*100.0}" upper="${pi*100.0}" />
+  </joint>
+  <joint name="$(arg prefix)joint1_drive" type="revolute">
+      <parent link="$(arg prefix)link_1"/>
+      <child link="$(arg prefix)link_1_wheel"/>
+      <origin xyz="0 0 -0.0825" rpy="0 0 0"/>
+      <axis xyz="0 1 0" />
+      <limit velocity="4.8" effort="1" lower="${-pi*100.0}" upper="${pi*100.0}" />
+  </joint>
+  <link name="$(arg prefix)link_1_wheel"/>
+  <link name="$(arg prefix)link_2"/>
+  <joint name="$(arg prefix)joint2_steer" type="revolute">
+      <parent link="$(arg prefix)base_link"/>
+      <child link="$(arg prefix)link_2"/>
+      <origin xyz="0.2135 -0.2554 0" rpy="0 0 0"/>
+      <axis xyz="0 0 1" />
+      <limit velocity="4.8" effort="1" lower="${-pi*100.0}" upper="${pi*100.0}" />
+  </joint>
+  <joint name="$(arg prefix)joint2_drive" type="revolute">
+      <parent link="$(arg prefix)link_2"/>
+      <child link="$(arg prefix)link_2_wheel"/>
+      <origin xyz="0 0 -0.0825" rpy="0 0 0"/>
+      <axis xyz="0 1 0" />
+      <limit velocity="4.8" effort="1" lower="${-pi*100.0}" upper="${pi*100.0}" />
+  </joint>
+  <link name="$(arg prefix)link_2_wheel"/>
+  <link name="$(arg prefix)link_3"/>
+  <joint name="$(arg prefix)joint3_steer" type="revolute">
+      <parent link="$(arg prefix)base_link"/>
+      <child link="$(arg prefix)link_3"/>
+      <origin xyz="-0.2135 0 0" rpy="0 0 0"/>
+      <axis xyz="0 0 1" />
+      <limit velocity="4.8" effort="1" lower="${-pi*100.0}" upper="${pi*100.0}" />
+  </joint>
+  <joint name="$(arg prefix)joint3_drive" type="revolute">
+      <parent link="$(arg prefix)link_3"/>
+      <child link="$(arg prefix)link_3_wheel"/>
+      <origin xyz="0 0 -0.0825" rpy="0 0 0"/>
+      <axis xyz="0 1 0" />
+      <limit velocity="4.8" effort="1" lower="${-pi*100.0}" upper="${pi*100.0}" />
+  </joint>
+  <link name="$(arg prefix)link_3_wheel"/>
   <xacro:ffw_sg2_follower_system
+    use_sim="$(arg use_sim)"
+    use_fake_hardware="$(arg use_fake_hardware)"
+    fake_sensor_commands="$(arg fake_sensor_commands)"/>
+  <xacro:ffw_sg2_base_system
     use_sim="$(arg use_sim)"
     use_fake_hardware="$(arg use_fake_hardware)"
