Commit message: Rename joints in ffw_sg2_base.ros2_control.xacro for clarity: changed 'joint2_steer' to 'right_wheel_steer' and 'joint2_drive' to 'right_wheel_drive'.

File: ffw_description/ros2_control/ffw_sg2_rev1_follower/ffw_sg2_base.ros2_control.xacro (robot description, xacro)
@@ -47,5 +47,5 @@
         <state_interface name="effort"/>
       </joint>
-      <joint name="joint2_steer">
+      <joint name="right_wheel_steer">
         <command_interface name="position"/>
         <state_interface name="position"/>
@@ -53,5 +53,5 @@
         <state_interface name="effort"/>
       </joint>
-      <joint name="joint2_drive">
+      <joint name="right_wheel_drive">
         <command_interface name="velocity"/>
         <state_interface name="position"/>

Commit message: Refactor swerve drive configuration and add new STL files for left and rear wheel components. Updated joint names for clarity in ffw_sg2_base.ros2_control.xacro and added lift link to URDF.

File: ffw_description/ros2_control/ffw_sg2_rev1_follower/ffw_sg2_base.ros2_control.xacro (robot description, xacro)
@@ -2,38 +2,44 @@
 <robot xmlns:xacro="http://www.ros.org/wiki/xacro">
   <xacro:macro name="ffw_sg2_base_system" params="use_sim:=^|false use_fake_hardware:=^|false fake_sensor_commands:=^|false">
-    <xacro:property name="initial_positions" value="${load_yaml(initial_positions_file)['initial_positions']}"/>
     <ros2_control name="ffw_sg2_base" type="system" is_async="true">
-      <hardware>
-        <plugin>dynamixel_hardware_interface/DynamixelHardware</plugin>
-        <param name="port_name">/dev/ttyUSB0</param>
-        <param name="baud_rate">4000000</param>
-        <param name="dynamixel_model_folder">/param/dxl_model</param>
-        <param name="number_of_joints">6</param>
-        <param name="number_of_transmissions">6</param>
-        <param name="disable_torque_at_init">true</param>
-        <param name="transmission_to_joint_matrix">
-          1, 0, 0, 0, 0, 0,
-          0, 1, 0, 0, 0, 0,
-          0, 0, 1, 0, 0, 0,
-          0, 0, 0, 1, 0, 0,
-          0, 0, 0, 0, 1, 0,
-          0, 0, 0, 0, 0, 1
-        </param>
-        <param name="joint_to_transmission_matrix">
-          1, 0, 0, 0, 0, 0,
-          0, 1, 0, 0, 0, 0,
-          0, 0, 1, 0, 0, 0,
-          0, 0, 0, 1, 0, 0,
-          0, 0, 0, 0, 1, 0,
-          0, 0, 0, 0, 0, 1
-        </param>
-        <param name="dynamixel_state_pub_msg_name">dynamixel_hardware_interface/dxl_state</param>
-        <param name="get_dynamixel_data_srv_name">dynamixel_hardware_interface/get_dxl_data</param>
-        <param name="set_dynamixel_data_srv_name">dynamixel_hardware_interface/set_dxl_data</param>
-        <param name="reboot_dxl_srv_name">dynamixel_hardware_interface/reboot_dxl</param>
-        <param name="set_dxl_torque_srv_name">dynamixel_hardware_interface/set_dxl_torque</param>
-        <param name="error_timeout_ms">500</param>
-      </hardware>
-      <joint name="joint1_steer">
+      <xacro:if value="$(arg use_sim)">
+        <hardware>
+          <plugin>gz_ros2_control/GazeboSimSystem</plugin>
+        </hardware>
+      </xacro:if>
+      <xacro:unless value="$(arg use_sim)">
+        <hardware>
+          <plugin>dynamixel_hardware_interface/DynamixelHardware</plugin>
+          <param name="port_name">/dev/ttyUSB0</param>
+          <param name="baud_rate">4000000</param>
+          <param name="dynamixel_model_folder">/param/dxl_model</param>
+          <param name="number_of_joints">6</param>
+          <param name="number_of_transmissions">6</param>
+          <param name="disable_torque_at_init">true</param>
+          <param name="transmission_to_joint_matrix">
+            1, 0, 0, 0, 0, 0,
+            0, 1, 0, 0, 0, 0,
+            0, 0, 1, 0, 0, 0,
+            0, 0, 0, 1, 0, 0,
+            0, 0, 0, 0, 1, 0,
+            0, 0, 0, 0, 0, 1
+          </param>
+          <param name="joint_to_transmission_matrix">
+            1, 0, 0, 0, 0, 0,
+            0, 1, 0, 0, 0, 0,
+            0, 0, 1, 0, 0, 0,
+            0, 0, 0, 1, 0, 0,
+            0, 0, 0, 0, 1, 0,
+            0, 0, 0, 0, 0, 1
+          </param>
+          <param name="dynamixel_state_pub_msg_name">dynamixel_hardware_interface/dxl_state</param>
+          <param name="get_dynamixel_data_srv_name">dynamixel_hardware_interface/get_dxl_data</param>
+          <param name="set_dynamixel_data_srv_name">dynamixel_hardware_interface/set_dxl_data</param>
+          <param name="reboot_dxl_srv_name">dynamixel_hardware_interface/reboot_dxl</param>
+          <param name="set_dxl_torque_srv_name">dynamixel_hardware_interface/set_dxl_torque</param>
+          <param name="error_timeout_ms">500</param>
+        </hardware>
+      </xacro:unless>
+      <joint name="left_wheel_steer">
         <command_interface name="position"/>
         <state_interface name="position"/>
@@ -41,5 +47,5 @@
         <state_interface name="effort"/>
       </joint>
-      <joint name="joint1_drive">
+      <joint name="left_wheel_drive">
         <command_interface name="velocity"/>
         <state_interface name="position"/>
@@ -59,5 +65,5 @@
         <state_interface name="effort"/>
       </joint>
-      <joint name="joint3_steer">
+      <joint name="rear_wheel_steer">
         <command_interface name="position"/>
         <state_interface name="position"/>
@@ -65,5 +71,5 @@
         <state_interface name="effort"/>
       </joint>
-      <joint name="joint3_drive">
+      <joint name="rear_wheel_drive">
         <command_interface name="velocity"/>
         <state_interface name="position"/>
@@ -71,5 +77,5 @@
         <state_interface name="effort"/>
       </joint>
-      <gpio name="dxl1_steer">
+      <gpio name="dxl1">
         <param name="type">virtual_dxl</param>
         <param name="ID">1</param>
@@ -92,5 +98,5 @@
         <param name="Profile Time">1000</param>
       </gpio>
-      <gpio name="dxl1_drive">
+      <gpio name="dxl2">
         <param name="type">virtual_dxl</param>
         <param name="ID">2</param>
@@ -114,5 +120,5 @@
         <param name="Profile Acceleration">100</param>
       </gpio>
-      <gpio name="dxl2_steer">
+      <gpio name="dxl3">
         <param name="type">virtual_dxl</param>
         <param name="ID">3</param>
@@ -135,5 +141,5 @@
         <param name="Profile Time">1000</param>
       </gpio>
-      <gpio name="dxl2_drive">
+      <gpio name="dxl4">
         <param name="type">virtual_dxl</param>
         <param name="ID">4</param>
@@ -157,5 +163,5 @@
         <param name="Profile Acceleration">100</param>
       </gpio>
-      <gpio name="dxl3_steer">
+      <gpio name="dxl5">
         <param name="type">virtual_dxl</param>
         <param name="ID">5</param>
@@ -178,5 +184,5 @@
         <param name="Profile Time">1000</param>
       </gpio>
-      <gpio name="dxl3_drive">
+      <gpio name="dxl6">
         <param name="type">virtual_dxl</param>
         <param name="ID">6</param>

File: ffw_description/urdf/ffw_sg2_rev1_follower/ffw_sg2_follower.urdf.xacro (robot description, xacro)
@@ -42,4 +42,26 @@
     </inertial>
   </link>
+  <link name="$(arg prefix)lift_link">
+    <visual>
+      <origin xyz="0 0 0" rpy="0 0 0" />
+      <geometry>
+        <mesh filename="${meshes_file_direction}/lift_link.stl" scale="0.001 0.001 0.001" />
+      </geometry>
+      <material name="silver">
+        <color rgba="0.75 0.75 0.75 1"/>
+      </material>
+    </visual>
+    <collision>
+      <origin xyz="0 0 0" rpy="0 0 0" />
+      <geometry>
+        <mesh filename="${meshes_file_direction}/lift_link.stl" scale="0.001 0.001 0.001" />
+      </geometry>
+    </collision>
+  </link>
+  <joint name="$(arg prefix)lift_fixed_joint" type="fixed">
+    <parent link="$(arg prefix)base_link"/>
+    <child link="$(arg prefix)lift_link"/>
+    <origin xyz="0.0 0.0 0.0" rpy="0 0 0"/>
+  </joint>
   <xacro:ffw_follower_body parent="$(arg prefix)base_link" prefix="$(arg prefix)">
     <origin xyz="0.0055 0 1.4316" rpy="0 0 0" />
@@ -51,20 +73,52 @@
     <origin xyz="0 0 -0.078" rpy="0 3.14159265359 0"/>
   </xacro:rh_p12_rn_a>
-  <link name="$(arg prefix)link_1"/>
-  <joint name="$(arg prefix)joint1_steer" type="revolute">
+  <link name="$(arg prefix)left_wheel_steer_link">
+    <visual>
+      <origin xyz="0 0 0" rpy="0 0 0" />
+      <geometry>
+        <mesh filename="${meshes_file_direction}/left_wheel_steer_link.stl" scale="0.001 0.001 0.001" />
+      </geometry>
+      <material name="silver">
+        <color rgba="0.75 0.75 0.75 1"/>
+      </material>
+    </visual>
+    <collision>
+      <origin xyz="0 0 0" rpy="0 0 0" />
+      <geometry>
+        <mesh filename="${meshes_file_direction}/left_wheel_steer_link.stl" scale="0.001 0.001 0.001" />
+      </geometry>
+    </collision>
+  </link>
+  <joint name="$(arg prefix)left_wheel_steer" type="revolute">
       <parent link="$(arg prefix)base_link"/>
-      <child link="$(arg prefix)link_1"/>
+      <child link="$(arg prefix)left_wheel_steer_link"/>
       <origin xyz="0.1371 0.2554 0.27555" rpy="0 0 0"/>
       <axis xyz="0 0 1" />
       <limit velocity="4.8" effort="1" lower="${-pi*6.0}" upper="${pi*6.0}" />
   </joint>
-  <joint name="$(arg prefix)joint1_drive" type="revolute">
-      <parent link="$(arg prefix)link_1"/>
-      <child link="$(arg prefix)link_1_wheel"/>
+  <joint name="$(arg prefix)left_wheel_drive" type="revolute">
+      <parent link="$(arg prefix)left_wheel_steer_link"/>
+      <child link="$(arg prefix)left_wheel_drive_link"/>
       <origin xyz="0 0 -0.18905" rpy="0 0 0"/>
       <axis xyz="0 1 0" />
       <limit velocity="4.8" effort="1" lower="${-pi*6.0}" upper="${pi*6.0}" />
   </joint>
-  <link name="$(arg prefix)link_1_wheel"/>
+  <link name="$(arg prefix)left_wheel_drive_link">
+    <visual>
+      <origin xyz="0 0 0" rpy="0 0 0" />
+      <geometry>
+        <mesh filename="${meshes_file_direction}/left_wheel_drive_link.stl" scale="0.001 0.001 0.001" />
+      </geometry>
+      <material name="silver">
+        <color rgba="0.75 0.75 0.75 1"/>
+      </material>
+    </visual>
+    <collision>
+      <origin xyz="0 0 0" rpy="0 0 0" />
+      <geometry>
+        <mesh filename="${meshes_file_direction}/left_wheel_drive_link.stl" scale="0.001 0.001 0.001" />
+      </geometry>
+    </collision>
+  </link>
   <joint name="$(arg prefix)right_wheel_steer" type="revolute">
       <parent link="$(arg prefix)base_link"/>
@@ -115,20 +169,52 @@
     </collision>
   </link>
-  <link name="$(arg prefix)link_3"/>
-  <joint name="$(arg prefix)joint3_steer" type="revolute">
+  <joint name="$(arg prefix)rear_wheel_steer" type="revolute">
       <parent link="$(arg prefix)base_link"/>
-      <child link="$(arg prefix)link_3"/>
+      <child link="$(arg prefix)rear_wheel_steer_link"/>
       <origin xyz="-0.2899 0 0.27555" rpy="0 0 0"/>
       <axis xyz="0 0 1" />
       <limit velocity="4.8" effort="1" lower="${-pi*6.0}" upper="${pi*6.0}" />
   </joint>
-  <joint name="$(arg prefix)joint3_drive" type="revolute">
-      <parent link="$(arg prefix)link_3"/>
-      <child link="$(arg prefix)link_3_wheel"/>
+  <link name="$(arg prefix)rear_wheel_steer_link">
+    <visual>
+      <origin xyz="0 0 0" rpy="0 0 0" />
+      <geometry>
+        <mesh filename="${meshes_file_direction}/rear_wheel_steer_link.stl" scale="0.001 0.001 0.001" />
+      </geometry>
+      <material name="silver">
+        <color rgba="0.75 0.75 0.75 1"/>
+      </material>
+    </visual>
+    <collision>
+      <origin xyz="0 0 0" rpy="0 0 0" />
+      <geometry>
+        <mesh filename="${meshes_file_direction}/rear_wheel_steer_link.stl" scale="0.001 0.001 0.001" />
+      </geometry>
+    </collision>
+  </link>
+  <joint name="$(arg prefix)rear_wheel_drive" type="revolute">
+      <parent link="$(arg prefix)rear_wheel_steer_link"/>
+      <child link="$(arg prefix)rear_wheel_drive_link"/>
       <origin xyz="0 0 -0.18905" rpy="0 0 0"/>
       <axis xyz="0 1 0" />
       <limit velocity="4.8" effort="1" lower="${-pi*6.0}" upper="${pi*6.0}" />
   </joint>
-  <link name="$(arg prefix)link_3_wheel"/>
+  <link name="$(arg prefix)rear_wheel_drive_link">
+    <visual>
+      <origin xyz="0 0 0" rpy="0 0 0" />
+      <geometry>
+        <mesh filename="${meshes_file_direction}/rear_wheel_drive_link.stl" scale="0.001 0.001 0.001" />
+      </geometry>
+      <material name="silver">
+        <color rgba="0.75 0.75 0.75 1"/>
+      </material>
+    </visual>
+    <collision>
+      <origin xyz="0 0 0" rpy="0 0 0" />
+      <geometry>
+        <mesh filename="${meshes_file_direction}/rear_wheel_drive_link.stl" scale="0.001 0.001 0.001" />
+      </geometry>
+    </collision>
+  </link>
   <xacro:ffw_sg2_follower_system
     use_sim="$(arg use_sim)"

Commit message: Update GPIO names and IDs in ffw_sg2_base.ros2_control.xacro for consistency; remove unnecessary whitespace in ffw_sg2_follower.ros2_control.xacro.

File: ffw_description/ros2_control/ffw_sg2_rev1_follower/ffw_sg2_base.ros2_control.xacro (robot description, xacro)
@@ -77,7 +77,7 @@
         <state_interface name="effort"/>
       </joint>
-      <gpio name="dxl1">
-        <param name="type">virtual_dxl</param>
-        <param name="ID">1</param>
+      <gpio name="dxl101">
+        <param name="type">virtual_dxl</param>
+        <param name="ID">101</param>
         <param name="model_num">620</param>
         <param name="comm_id">200</param>
@@ -98,7 +98,7 @@
         <param name="Profile Time">1000</param>
       </gpio>
-      <gpio name="dxl2">
-        <param name="type">virtual_dxl</param>
-        <param name="ID">2</param>
+      <gpio name="dxl102">
+        <param name="type">virtual_dxl</param>
+        <param name="ID">102</param>
         <param name="model_num">623</param>
         <param name="comm_id">200</param>
@@ -120,7 +120,7 @@
         <param name="Profile Acceleration">100</param>
       </gpio>
-      <gpio name="dxl3">
-        <param name="type">virtual_dxl</param>
-        <param name="ID">3</param>
+      <gpio name="dxl103">
+        <param name="type">virtual_dxl</param>
+        <param name="ID">103</param>
         <param name="model_num">621</param>
         <param name="comm_id">200</param>
@@ -141,7 +141,7 @@
         <param name="Profile Time">1000</param>
       </gpio>
-      <gpio name="dxl4">
-        <param name="type">virtual_dxl</param>
-        <param name="ID">4</param>
+      <gpio name="dxl104">
+        <param name="type">virtual_dxl</param>
+        <param name="ID">104</param>
         <param name="model_num">624</param>
         <param name="comm_id">200</param>
@@ -163,7 +163,7 @@
         <param name="Profile Acceleration">100</param>
       </gpio>
-      <gpio name="dxl5">
-        <param name="type">virtual_dxl</param>
-        <param name="ID">5</param>
+      <gpio name="dxl105">
+        <param name="type">virtual_dxl</param>
+        <param name="ID">105</param>
         <param name="model_num">622</param>
         <param name="comm_id">200</param>
@@ -184,7 +184,7 @@
         <param name="Profile Time">1000</param>
       </gpio>
-      <gpio name="dxl6">
-        <param name="type">virtual_dxl</param>
-        <param name="ID">6</param>
+      <gpio name="dxl106">
+        <param name="type">virtual_dxl</param>
+        <param name="ID">106</param>
         <param name="model_num">625</param>
         <param name="comm_id">200</param>

File: ffw_description/ros2_control/ffw_sg2_rev1_follower/ffw_sg2_follower.ros2_control.xacro (robot description, xacro)
@@ -2,5 +2,4 @@
 <robot xmlns:xacro="http://www.ros.org/wiki/xacro">
   <xacro:macro name="ffw_sg2_follower_system" params="use_sim:=^|false use_fake_hardware:=^|false fake_sensor_commands:=^|false">
-    <xacro:property name="initial_positions" value="${load_yaml(initial_positions_file)['initial_positions']}"/>
     <ros2_control name="ffw_sg2_follower" type="system" is_async="true">
       <xacro:if value="$(arg use_sim)">
