Commit message: fix: Moved swerve dxl into main dhi config due to hardware changes

File: ffw_description/ros2_control/ffw_sg2_rev1_follower/ffw_sg2_base.ros2_control.xacro (robot description, xacro)
@@ -10,49 +10,38 @@
       <xacro:unless value="$(arg use_sim)">
         <hardware>
-          <plugin>dynamixel_hardware_interface/DynamixelHardware</plugin>
-          <param name="port_name">/dev/ttyUSB0</param>
-          <param name="baud_rate">4000000</param>
-          <param name="dynamixel_model_folder">/param/dxl_model</param>
-          <param name="number_of_joints">6</param>
-          <param name="number_of_transmissions">6</param>
-          <param name="disable_torque_at_init">true</param>
-          <param name="transmission_to_joint_matrix">
-            1, 0, 0, 0, 0, 0,
-            0, 1, 0, 0, 0, 0,
-            0, 0, 1, 0, 0, 0,
-            0, 0, 0, 1, 0, 0,
-            0, 0, 0, 0, 1, 0,
-            0, 0, 0, 0, 0, 1
-          </param>
-          <param name="joint_to_transmission_matrix">
-            1, 0, 0, 0, 0, 0,
-            0, 1, 0, 0, 0, 0,
-            0, 0, 1, 0, 0, 0,
-            0, 0, 0, 1, 0, 0,
-            0, 0, 0, 0, 1, 0,
-            0, 0, 0, 0, 0, 1
-          </param>
-          <param name="dynamixel_state_pub_msg_name">dynamixel_hardware_interface/dxl_state</param>
-          <param name="get_dynamixel_data_srv_name">dynamixel_hardware_interface/get_dxl_data</param>
-          <param name="set_dynamixel_data_srv_name">dynamixel_hardware_interface/set_dxl_data</param>
-          <param name="reboot_dxl_srv_name">dynamixel_hardware_interface/reboot_dxl</param>
-          <param name="set_dxl_torque_srv_name">dynamixel_hardware_interface/set_dxl_torque</param>
-          <param name="error_timeout_ms">500</param>
+          <xacro:if value="${use_fake_hardware}">
+            <plugin>fake_components/GenericSystem</plugin>
+            <param name="fake_sensor_commands">${fake_sensor_commands}</param>
+            <param name="state_following_offset">0.0</param>
+          </xacro:if>
+          <xacro:unless value="${use_fake_hardware}">
+            <plugin>dynamixel_hardware_interface/DynamixelHardware</plugin>
+            <param name="port_name">/dev/ttyUSB0</param>
+            <param name="baud_rate">4000000</param>
+            <param name="dynamixel_model_folder">/param/dxl_model</param>
+            <param name="number_of_joints">3</param>
+            <param name="number_of_transmissions">3</param>
+            <param name="disable_torque_at_init">true</param>
+            <param name="transmission_to_joint_matrix">
+              1, 0, 0,
+              0, 1, 0,
+              0, 0, 1
+            </param>
+            <param name="joint_to_transmission_matrix">
+              1, 0, 0,
+              0, 1, 0,
+              0, 0, 1
+            </param>
+            <param name="dynamixel_state_pub_msg_name">dynamixel_hardware_interface/dxl_state</param>
+            <param name="get_dynamixel_data_srv_name">dynamixel_hardware_interface/get_dxl_data</param>
+            <param name="set_dynamixel_data_srv_name">dynamixel_hardware_interface/set_dxl_data</param>
+            <param name="reboot_dxl_srv_name">dynamixel_hardware_interface/reboot_dxl</param>
+            <param name="set_dxl_torque_srv_name">dynamixel_hardware_interface/set_dxl_torque</param>
+            <param name="error_timeout_ms">500</param>
+          </xacro:unless>
         </hardware>
       </xacro:unless>
-      <joint name="left_wheel_steer">
-        <command_interface name="position"/>
-        <state_interface name="position"/>
-        <state_interface name="velocity"/>
-        <state_interface name="effort"/>
-      </joint>
       <joint name="left_wheel_drive">
         <command_interface name="velocity"/>
-        <state_interface name="position"/>
-        <state_interface name="velocity"/>
-        <state_interface name="effort"/>
-      </joint>
-      <joint name="right_wheel_steer">
-        <command_interface name="position"/>
         <state_interface name="position"/>
         <state_interface name="velocity"/>
@@ -65,10 +54,4 @@
         <state_interface name="effort"/>
       </joint>
-      <joint name="rear_wheel_steer">
-        <command_interface name="position"/>
-        <state_interface name="position"/>
-        <state_interface name="velocity"/>
-        <state_interface name="effort"/>
-      </joint>
       <joint name="rear_wheel_drive">
         <command_interface name="velocity"/>
@@ -77,25 +60,4 @@
         <state_interface name="effort"/>
       </joint>
-      <gpio name="dxl101">
-        <param name="type">virtual_dxl</param>
-        <param name="ID">101</param>
-        <param name="model_num">620</param>
-        <param name="comm_id">200</param>
-        <command_interface name="Goal Position"/>
-        <state_interface name="Present Current"/>
-        <state_interface name="Present Velocity"/>
-        <state_interface name="Present Position"/>
-        <param name="Drive Mode">5</param>
-        <param name="Operating Mode">3</param>
-        <param name="Velocity Limit">12592</param>
-        <param name="Acceleration Limit">125920</param>
-        <param name="Min Position Limit">-1572864</param>
-        <param name="Max Position Limit">1572864</param>
-        <param name="Return Delay Time">0</param>
-        <param name="Profile Velocity">12592</param>
-        <param name="Profile Acceleration">12592</param>
-        <param name="Profile Acceleration Time">300</param>
-        <param name="Profile Time">1000</param>
-      </gpio>
       <gpio name="dxl102">
         <param name="type">virtual_dxl</param>
@@ -120,25 +82,4 @@
         <param name="Profile Acceleration">100</param>
       </gpio>
-      <gpio name="dxl103">
-        <param name="type">virtual_dxl</param>
-        <param name="ID">103</param>
-        <param name="model_num">621</param>
-        <param name="comm_id">200</param>
-        <command_interface name="Goal Position"/>
-        <state_interface name="Present Current"/>
-        <state_interface name="Present Velocity"/>
-        <state_interface name="Present Position"/>
-        <param name="Drive Mode">5</param>
-        <param name="Operating Mode">3</param>
-        <param name="Velocity Limit">12592</param>
-        <param name="Acceleration Limit">125920</param>
-        <param name="Min Position Limit">-1572864</param>
-        <param name="Max Position Limit">1572864</param>
-        <param name="Return Delay Time">0</param>
-        <param name="Profile Velocity">12592</param>
-        <param name="Profile Acceleration">12592</param>
-        <param name="Profile Acceleration Time">300</param>
-        <param name="Profile Time">1000</param>
-      </gpio>
       <gpio name="dxl104">
         <param name="type">virtual_dxl</param>
@@ -162,25 +103,4 @@
         <param name="Velocity FF Gain">50000</param>
         <param name="Profile Acceleration">100</param>
-      </gpio>
-      <gpio name="dxl105">
-        <param name="type">virtual_dxl</param>
-        <param name="ID">105</param>
-        <param name="model_num">622</param>
-        <param name="comm_id">200</param>
-        <command_interface name="Goal Position"/>
-        <state_interface name="Present Current"/>
-        <state_interface name="Present Velocity"/>
-        <state_interface name="Present Position"/>
-        <param name="Drive Mode">5</param>
-        <param name="Operating Mode">3</param>
-        <param name="Velocity Limit">12592</param>
-        <param name="Acceleration Limit">125920</param>
-        <param name="Min Position Limit">-1572864</param>
-        <param name="Max Position Limit">1572864</param>
-        <param name="Return Delay Time">0</param>
-        <param name="Profile Velocity">12592</param>
-        <param name="Profile Acceleration">12592</param>
-        <param name="Profile Acceleration Time">300</param>
-        <param name="Profile Time">1000</param>
       </gpio>
       <gpio name="dxl106">

File: ffw_description/ros2_control/ffw_sg2_rev1_follower/ffw_sg2_follower.ros2_control.xacro (robot description, xacro)
@@ -20,48 +20,54 @@
             <param name="baud_rate">4000000</param>
             <param name="dynamixel_model_folder">/param/dxl_model</param>
-            <param name="number_of_joints">19</param>
-            <param name="number_of_transmissions">19</param>
+            <param name="number_of_joints">22</param>
+            <param name="number_of_transmissions">22</param>
             <param name="disable_torque_at_init">true</param>
             <param name="transmission_to_joint_matrix">
-              1, 0, 0, 0, 0, 0, 0, 0, 0, 0, 0, 0, 0, 0, 0, 0, 0, 0, 0,
-              0, 1, 0, 0, 0, 0, 0, 0, 0, 0, 0, 0, 0, 0, 0, 0, 0, 0, 0,
-              0, 0, 1, 0, 0, 0, 0, 0, 0, 0, 0, 0, 0, 0, 0, 0, 0, 0, 0,
-              0, 0, 0, 1, 0, 0, 0, 0, 0, 0, 0, 0, 0, 0, 0, 0, 0, 0, 0,
-              0, 0, 0, 0, 1, 0, 0, 0, 0, 0, 0, 0, 0, 0, 0, 0, 0, 0, 0,
-              0, 0, 0, 0, 0, 1, 0, 0, 0, 0, 0, 0, 0, 0, 0, 0, 0, 0, 0,
-              0, 0, 0, 0, 0, 0, 1, 0, 0, 0, 0, 0, 0, 0, 0, 0, 0, 0, 0,
-              0, 0, 0, 0, 0, 0, 0, 1, 0, 0, 0, 0, 0, 0, 0, 0, 0, 0, 0,
-              0, 0, 0, 0, 0, 0, 0, 0, 1, 0, 0, 0, 0, 0, 0, 0, 0, 0, 0,
-              0, 0, 0, 0, 0, 0, 0, 0, 0, 1, 0, 0, 0, 0, 0, 0, 0, 0, 0,
-              0, 0, 0, 0, 0, 0, 0, 0, 0, 0, 1, 0, 0, 0, 0, 0, 0, 0, 0,
-              0, 0, 0, 0, 0, 0, 0, 0, 0, 0, 0, 1, 0, 0, 0, 0, 0, 0, 0,
-              0, 0, 0, 0, 0, 0, 0, 0, 0, 0, 0, 0, 1, 0, 0, 0, 0, 0, 0,
-              0, 0, 0, 0, 0, 0, 0, 0, 0, 0, 0, 0, 0, 1, 0, 0, 0, 0, 0,
-              0, 0, 0, 0, 0, 0, 0, 0, 0, 0, 0, 0, 0, 0, 1, 0, 0, 0, 0,
-              0, 0, 0, 0, 0, 0, 0, 0, 0, 0, 0, 0, 0, 0, 0, 1, 0, 0, 0,
-              0, 0, 0, 0, 0, 0, 0, 0, 0, 0, 0, 0, 0, 0, 0, 0, 1, 0, 0,
-              0, 0, 0, 0, 0, 0, 0, 0, 0, 0, 0, 0, 0, 0, 0, 0, 0, 1, 0,
-              0, 0, 0, 0, 0, 0, 0, 0, 0, 0, 0, 0, 0, 0, 0, 0, 0, 0, 1
+              1, 0, 0, 0, 0, 0, 0, 0, 0, 0, 0, 0, 0, 0, 0, 0, 0, 0, 0, 0, 0, 0,
+              0, 1, 0, 0, 0, 0, 0, 0, 0, 0, 0, 0, 0, 0, 0, 0, 0, 0, 0, 0, 0, 0,
+              0, 0, 1, 0, 0, 0, 0, 0, 0, 0, 0, 0, 0, 0, 0, 0, 0, 0, 0, 0, 0, 0,
+              0, 0, 0, 1, 0, 0, 0, 0, 0, 0, 0, 0, 0, 0, 0, 0, 0, 0, 0, 0, 0, 0,
+              0, 0, 0, 0, 1, 0, 0, 0, 0, 0, 0, 0, 0, 0, 0, 0, 0, 0, 0, 0, 0, 0,
+              0, 0, 0, 0, 0, 1, 0, 0, 0, 0, 0, 0, 0, 0, 0, 0, 0, 0, 0, 0, 0, 0,
+              0, 0, 0, 0, 0, 0, 1, 0, 0, 0, 0, 0, 0, 0, 0, 0, 0, 0, 0, 0, 0, 0,
+              0, 0, 0, 0, 0, 0, 0, 1, 0, 0, 0, 0, 0, 0, 0, 0, 0, 0, 0, 0, 0, 0,
+              0, 0, 0, 0, 0, 0, 0, 0, 1, 0, 0, 0, 0, 0, 0, 0, 0, 0, 0, 0, 0, 0,
+              0, 0, 0, 0, 0, 0, 0, 0, 0, 1, 0, 0, 0, 0, 0, 0, 0, 0, 0, 0, 0, 0,
+              0, 0, 0, 0, 0, 0, 0, 0, 0, 0, 1, 0, 0, 0, 0, 0, 0, 0, 0, 0, 0, 0,
+              0, 0, 0, 0, 0, 0, 0, 0, 0, 0, 0, 1, 0, 0, 0, 0, 0, 0, 0, 0, 0, 0,
+              0, 0, 0, 0, 0, 0, 0, 0, 0, 0, 0, 0, 1, 0, 0, 0, 0, 0, 0, 0, 0, 0,
+              0, 0, 0, 0, 0, 0, 0, 0, 0, 0, 0, 0, 0, 1, 0, 0, 0, 0, 0, 0, 0, 0,
+              0, 0, 0, 0, 0, 0, 0, 0, 0, 0, 0, 0, 0, 0, 1, 0, 0, 0, 0, 0, 0, 0,
+              0, 0, 0, 0, 0, 0, 0, 0, 0, 0, 0, 0, 0, 0, 0, 1, 0, 0, 0, 0, 0, 0,
+              0, 0, 0, 0, 0, 0, 0, 0, 0, 0, 0, 0, 0, 0, 0, 0, 1, 0, 0, 0, 0, 0,
+              0, 0, 0, 0, 0, 0, 0, 0, 0, 0, 0, 0, 0, 0, 0, 0, 0, 1, 0, 0, 0, 0,
+              0, 0, 0, 0, 0, 0, 0, 0, 0, 0, 0, 0, 0, 0, 0, 0, 0, 0, 1, 0, 0, 0,
+              0, 0, 0, 0, 0, 0, 0, 0, 0, 0, 0, 0, 0, 0, 0, 0, 0, 0, 0, 1, 0, 0,
+              0, 0, 0, 0, 0, 0, 0, 0, 0, 0, 0, 0, 0, 0, 0, 0, 0, 0, 0, 0, 1, 0,
+              0, 0, 0, 0, 0, 0, 0, 0, 0, 0, 0, 0, 0, 0, 0, 0, 0, 0, 0, 0, 0, 1
             </param>
             <param name="joint_to_transmission_matrix">
-              1, 0, 0, 0, 0, 0, 0, 0, 0, 0, 0, 0, 0, 0, 0, 0, 0, 0, 0,
-              0, 1, 0, 0, 0, 0, 0, 0, 0, 0, 0, 0, 0, 0, 0, 0, 0, 0, 0,
-              0, 0, 1, 0, 0, 0, 0, 0, 0, 0, 0, 0, 0, 0, 0, 0, 0, 0, 0,
-              0, 0, 0, 1, 0, 0, 0, 0, 0, 0, 0, 0, 0, 0, 0, 0, 0, 0, 0,
-              0, 0, 0, 0, 1, 0, 0, 0, 0, 0, 0, 0, 0, 0, 0, 0, 0, 0, 0,
-              0, 0, 0, 0, 0, 1, 0, 0, 0, 0, 0, 0, 0, 0, 0, 0, 0, 0, 0,
-              0, 0, 0, 0, 0, 0, 1, 0, 0, 0, 0, 0, 0, 0, 0, 0, 0, 0, 0,
-              0, 0, 0, 0, 0, 0, 0, 1, 0, 0, 0, 0, 0, 0, 0, 0, 0, 0, 0,
-              0, 0, 0, 0, 0, 0, 0, 0, 1, 0, 0, 0, 0, 0, 0, 0, 0, 0, 0,
-              0, 0, 0, 0, 0, 0, 0, 0, 0, 1, 0, 0, 0, 0, 0, 0, 0, 0, 0,
-              0, 0, 0, 0, 0, 0, 0, 0, 0, 0, 1, 0, 0, 0, 0, 0, 0, 0, 0,
-              0, 0, 0, 0, 0, 0, 0, 0, 0, 0, 0, 1, 0, 0, 0, 0, 0, 0, 0,
-              0, 0, 0, 0, 0, 0, 0, 0, 0, 0, 0, 0, 1, 0, 0, 0, 0, 0, 0,
-              0, 0, 0, 0, 0, 0, 0, 0, 0, 0, 0, 0, 0, 1, 0, 0, 0, 0, 0,
-              0, 0, 0, 0, 0, 0, 0, 0, 0, 0, 0, 0, 0, 0, 1, 0, 0, 0, 0,
-              0, 0, 0, 0, 0, 0, 0, 0, 0, 0, 0, 0, 0, 0, 0, 1, 0, 0, 0,
-              0, 0, 0, 0, 0, 0, 0, 0, 0, 0, 0, 0, 0, 0, 0, 0, 1, 0, 0,
-              0, 0, 0, 0, 0, 0, 0, 0, 0, 0, 0, 0, 0, 0, 0, 0, 0, 1, 0,
-              0, 0, 0, 0, 0, 0, 0, 0, 0, 0, 0, 0, 0, 0, 0, 0, 0, 0, 1
+              1, 0, 0, 0, 0, 0, 0, 0, 0, 0, 0, 0, 0, 0, 0, 0, 0, 0, 0, 0, 0, 0,
+              0, 1, 0, 0, 0, 0, 0, 0, 0, 0, 0, 0, 0, 0, 0, 0, 0, 0, 0, 0, 0, 0,
+              0, 0, 1, 0, 0, 0, 0, 0, 0, 0, 0, 0, 0, 0, 0, 0, 0, 0, 0, 0, 0, 0,
+              0, 0, 0, 1, 0, 0, 0, 0, 0, 0, 0, 0, 0, 0, 0, 0, 0, 0, 0, 0, 0, 0,
+              0, 0, 0, 0, 1, 0, 0, 0, 0, 0, 0, 0, 0, 0, 0, 0, 0, 0, 0, 0, 0, 0,
+              0, 0, 0, 0, 0, 1, 0, 0, 0, 0, 0, 0, 0, 0, 0, 0, 0, 0, 0, 0, 0, 0,
+              0, 0, 0, 0, 0, 0, 1, 0, 0, 0, 0, 0, 0, 0, 0, 0, 0, 0, 0, 0, 0, 0,
+              0, 0, 0, 0, 0, 0, 0, 1, 0, 0, 0, 0, 0, 0, 0, 0, 0, 0, 0, 0, 0, 0,
+              0, 0, 0, 0, 0, 0, 0, 0, 1, 0, 0, 0, 0, 0, 0, 0, 0, 0, 0, 0, 0, 0,
+              0, 0, 0, 0, 0, 0, 0, 0, 0, 1, 0, 0, 0, 0, 0, 0, 0, 0, 0, 0, 0, 0,
+              0, 0, 0, 0, 0, 0, 0, 0, 0, 0, 1, 0, 0, 0, 0, 0, 0, 0, 0, 0, 0, 0,
+              0, 0, 0, 0, 0, 0, 0, 0, 0, 0, 0, 1, 0, 0, 0, 0, 0, 0, 0, 0, 0, 0,
+              0, 0, 0, 0, 0, 0, 0, 0, 0, 0, 0, 0, 1, 0, 0, 0, 0, 0, 0, 0, 0, 0,
+              0, 0, 0, 0, 0, 0, 0, 0, 0, 0, 0, 0, 0, 1, 0, 0, 0, 0, 0, 0, 0, 0,
+              0, 0, 0, 0, 0, 0, 0, 0, 0, 0, 0, 0, 0, 0, 1, 0, 0, 0, 0, 0, 0, 0,
+              0, 0, 0, 0, 0, 0, 0, 0, 0, 0, 0, 0, 0, 0, 0, 1, 0, 0, 0, 0, 0, 0,
+              0, 0, 0, 0, 0, 0, 0, 0, 0, 0, 0, 0, 0, 0, 0, 0, 1, 0, 0, 0, 0, 0,
+              0, 0, 0, 0, 0, 0, 0, 0, 0, 0, 0, 0, 0, 0, 0, 0, 0, 1, 0, 0, 0, 0,
+              0, 0, 0, 0, 0, 0, 0, 0, 0, 0, 0, 0, 0, 0, 0, 0, 0, 0, 1, 0, 0, 0,
+              0, 0, 0, 0, 0, 0, 0, 0, 0, 0, 0, 0, 0, 0, 0, 0, 0, 0, 0, 1, 0, 0,
+              0, 0, 0, 0, 0, 0, 0, 0, 0, 0, 0, 0, 0, 0, 0, 0, 0, 0, 0, 0, 1, 0,
+              0, 0, 0, 0, 0, 0, 0, 0, 0, 0, 0, 0, 0, 0, 0, 0, 0, 0, 0, 0, 0, 1
             </param>
             <param name="dynamixel_state_pub_msg_name">dynamixel_hardware_interface/dxl_state</param>
@@ -168,4 +174,22 @@
         <state_interface name="velocity"/>
       </joint>
+      <joint name="left_wheel_steer">
+        <command_interface name="position"/>
+        <state_interface name="position"/>
+        <state_interface name="velocity"/>
+        <state_interface name="effort"/>
+      </joint>
+      <joint name="right_wheel_steer">
+        <command_interface name="position"/>
+        <state_interface name="position"/>
+        <state_interface name="velocity"/>
+        <state_interface name="effort"/>
+      </joint>
+      <joint name="rear_wheel_steer">
+        <command_interface name="position"/>
+        <state_interface name="position"/>
+        <state_interface name="velocity"/>
+        <state_interface name="effort"/>
+      </joint>
       <!-- RIGHT ARM -->
       <gpio name="dxl1">
@@ -541,4 +565,64 @@
         <param name="Feedforward 2nd Gain">30</param>
       </gpio>
+      <!-- LEFT WHEEL -->
+      <gpio name="dxl101">
+        <param name="type">dxl</param>
+        <param name="ID">101</param>
+        <command_interface name="Goal Position"/>
+        <state_interface name="Present Current"/>
+        <state_interface name="Present Velocity"/>
+        <state_interface name="Present Position"/>
+        <param name="Drive Mode">5</param>
+        <param name="Operating Mode">3</param>
+        <param name="Velocity Limit">12592</param>
+        <param name="Acceleration Limit">125920</param>
+        <param name="Min Position Limit">-1572864</param>
+        <param name="Max Position Limit">1572864</param>
+        <param name="Return Delay Time">0</param>
+        <param name="Profile Velocity">12592</param>
+        <param name="Profile Acceleration">12592</param>
+        <param name="Profile Acceleration Time">300</param>
+        <param name="Profile Time">1000</param>
+      </gpio>
+      <!-- RIGHT WHEEL -->
+      <gpio name="dxl103">
+        <param name="type">dxl</param>
+        <param name="ID">103</param>
+        <command_interface name="Goal Position"/>
+        <state_interface name="Present Current"/>
+        <state_interface name="Present Velocity"/>
+        <state_interface name="Present Position"/>
+        <param name="Drive Mode">5</param>
+        <param name="Operating Mode">3</param>
+        <param name="Velocity Limit">12592</param>
+        <param name="Acceleration Limit">125920</param>
+        <param name="Min Position Limit">-1572864</param>
+        <param name="Max Position Limit">1572864</param>
+        <param name="Return Delay Time">0</param>
+        <param name="Profile Velocity">12592</param>
+        <param name="Profile Acceleration">12592</param>
+        <param name="Profile Acceleration Time">300</param>
+        <param name="Profile Time">1000</param>
+      </gpio>
+      <!-- REAR WHEEL -->
+      <gpio name="dxl105">
+        <param name="type">dxl</param>
+        <param name="ID">105</param>
+        <command_interface name="Goal Position"/>
+        <state_interface name="Present Current"/>
+        <state_interface name="Present Velocity"/>
+        <state_interface name="Present Position"/>
+        <param name="Drive Mode">5</param>
+        <param name="Operating Mode">3</param>
+        <param name="Velocity Limit">12592</param>
+        <param name="Acceleration Limit">125920</param>
+        <param name="Min Position Limit">-1572864</param>
+        <param name="Max Position Limit">1572864</param>
+        <param name="Return Delay Time">0</param>
+        <param name="Profile Velocity">12592</param>
+        <param name="Profile Acceleration">12592</param>
+        <param name="Profile Acceleration Time">300</param>
+        <param name="Profile Time">1000</param>
+      </gpio>
     </ros2_control>
   </xacro:macro>
