Commit message: Update URDF and add new STL files for right wheel components

File: ffw_description/urdf/ffw_sg2_rev1_follower/ffw_sg2_follower.urdf.xacro (robot description, xacro)
@@ -55,46 +55,78 @@
       <parent link="$(arg prefix)base_link"/>
       <child link="$(arg prefix)link_1"/>
-      <origin xyz="0.2135 0.2554 0" rpy="0 0 0"/>
+      <origin xyz="0.1371 0.2554 0.27555" rpy="0 0 0"/>
       <axis xyz="0 0 1" />
-      <limit velocity="4.8" effort="1" lower="${-pi*100.0}" upper="${pi*100.0}" />
+      <limit velocity="4.8" effort="1" lower="${-pi*6.0}" upper="${pi*6.0}" />
   </joint>
   <joint name="$(arg prefix)joint1_drive" type="revolute">
       <parent link="$(arg prefix)link_1"/>
       <child link="$(arg prefix)link_1_wheel"/>
-      <origin xyz="0 0 -0.0825" rpy="0 0 0"/>
+      <origin xyz="0 0 -0.18905" rpy="0 0 0"/>
       <axis xyz="0 1 0" />
-      <limit velocity="4.8" effort="1" lower="${-pi*100.0}" upper="${pi*100.0}" />
+      <limit velocity="4.8" effort="1" lower="${-pi*6.0}" upper="${pi*6.0}" />
   </joint>
   <link name="$(arg prefix)link_1_wheel"/>
-  <link name="$(arg prefix)link_2"/>
-  <joint name="$(arg prefix)joint2_steer" type="revolute">
+  <joint name="$(arg prefix)right_wheel_steer" type="revolute">
       <parent link="$(arg prefix)base_link"/>
-      <child link="$(arg prefix)link_2"/>
-      <origin xyz="0.2135 -0.2554 0" rpy="0 0 0"/>
+      <child link="$(arg prefix)right_wheel_steer_link"/>
+      <origin xyz="0.1371 -0.2554 0.27555" rpy="0 0 0"/>
       <axis xyz="0 0 1" />
-      <limit velocity="4.8" effort="1" lower="${-pi*100.0}" upper="${pi*100.0}" />
+      <limit velocity="4.8" effort="1" lower="${-pi*6.0}" upper="${pi*6.0}" />
   </joint>
-  <joint name="$(arg prefix)joint2_drive" type="revolute">
-      <parent link="$(arg prefix)link_2"/>
-      <child link="$(arg prefix)link_2_wheel"/>
-      <origin xyz="0 0 -0.0825" rpy="0 0 0"/>
+  <link name="$(arg prefix)right_wheel_steer_link">
+    <visual>
+      <origin xyz="0 0 0" rpy="0 0 0" />
+      <geometry>
+        <mesh filename="${meshes_file_direction}/right_wheel_steer_link.stl" scale="0.001 0.001 0.001" />
+      </geometry>
+      <material name="silver">
+        <color rgba="0.75 0.75 0.75 1"/>
+      </material>
+    </visual>
+    <collision>
+      <origin xyz="0 0 0" rpy="0 0 0" />
+      <geometry>
+        <mesh filename="${meshes_file_direction}/right_wheel_steer_link.stl" scale="0.001 0.001 0.001" />
+      </geometry>
+    </collision>
+  </link>
+  <joint name="$(arg prefix)right_wheel_drive" type="revolute">
+      <parent link="$(arg prefix)right_wheel_steer_link"/>
+      <child link="$(arg prefix)right_wheel_drive_link"/>
+      <origin xyz="0 0 -0.18905" rpy="0 0 0"/>
       <axis xyz="0 1 0" />
-      <limit velocity="4.8" effort="1" lower="${-pi*100.0}" upper="${pi*100.0}" />
+      <limit velocity="4.8" effort="1" lower="${-pi*6.0}" upper="${pi*6.0}" />
   </joint>
-  <link name="$(arg prefix)link_2_wheel"/>
+  <link name="$(arg prefix)right_wheel_drive_link">
+    <visual>
+      <origin xyz="0 0 0" rpy="0 0 0" />
+      <geometry>
+        <mesh filename="${meshes_file_direction}/right_wheel_drive_link.stl" scale="0.001 0.001 0.001" />
+      </geometry>
+      <material name="silver">
+        <color rgba="0.75 0.75 0.75 1"/>
+      </material>
+    </visual>
+    <collision>
+      <origin xyz="0 0 0" rpy="0 0 0" />
+      <geometry>
+        <mesh filename="${meshes_file_direction}/right_wheel_drive_link.stl" scale="0.001 0.001 0.001" />
+      </geometry>
+    </collision>
+  </link>
   <link name="$(arg prefix)link_3"/>
   <joint name="$(arg prefix)joint3_steer" type="revolute">
       <parent link="$(arg prefix)base_link"/>
       <child link="$(arg prefix)link_3"/>
-      <origin xyz="-0.2135 0 0" rpy="0 0 0"/>
+      <origin xyz="-0.2899 0 0.27555" rpy="0 0 0"/>
       <axis xyz="0 0 1" />
-      <limit velocity="4.8" effort="1" lower="${-pi*100.0}" upper="${pi*100.0}" />
+      <limit velocity="4.8" effort="1" lower="${-pi*6.0}" upper="${pi*6.0}" />
   </joint>
   <joint name="$(arg prefix)joint3_drive" type="revolute">
       <parent link="$(arg prefix)link_3"/>
       <child link="$(arg prefix)link_3_wheel"/>
-      <origin xyz="0 0 -0.0825" rpy="0 0 0"/>
+      <origin xyz="0 0 -0.18905" rpy="0 0 0"/>
       <axis xyz="0 1 0" />
-      <limit velocity="4.8" effort="1" lower="${-pi*100.0}" upper="${pi*100.0}" />
+      <limit velocity="4.8" effort="1" lower="${-pi*6.0}" upper="${pi*6.0}" />
   </joint>
   <link name="$(arg prefix)link_3_wheel"/>

Commit message: fix: Adjust follower body origin position in URDF to correct alignment

File: ffw_description/urdf/ffw_sg2_rev1_follower/ffw_sg2_follower.urdf.xacro (robot description, xacro)
@@ -65,5 +65,5 @@
   </joint>
   <xacro:ffw_follower_body parent="$(arg prefix)base_link" prefix="$(arg prefix)">
-    <origin xyz="0.0055 0 1.4316" rpy="0 0 0" />
+    <origin xyz="-0.0199 0 1.4316" rpy="0 0 0" />
   </xacro:ffw_follower_body>
   <xacro:rh_p12_rn_a parent="$(arg prefix)arm_l_link7" prefix="$(arg prefix)gripper_l_">

Commit message: feat: Add launch file and URDF intertia for sg2_rev1

File: ffw_description/urdf/ffw_sg2_rev1_follower/ffw_sg2_follower.urdf.xacro (robot description, xacro)
@@ -35,9 +35,9 @@
     </collision>
     <inertial>
-      <origin xyz="-8.880608700e-03 -4.758427800e-03 3.886366400e-01" />
-      <mass value="5.435831600e+01" />
-      <inertia ixx="1.188633900e+06" ixy="6.334393100e+02" ixz="-1.454811600e+05"
-      iyy="1.090949100e+06" iyz="-5.126785200e+03"
-      izz="4.492808000e+05" />
+       <origin xyz="-4.574796400e-02 6.581058800e-03 1.943184200e-01" />
+       <mass value="3.598943900e+01" />
+       <inertia ixx="1.725473500e+04" ixy="6.471795500e-02" ixz="1.890204600e-01"
+       iyy="3.983747500e+04" iyz="1.716567300e-01"
+       izz="2.846139500e+04" />
     </inertial>
   </link>
@@ -58,4 +58,11 @@
       </geometry>
     </collision>
+    <inertial>
+       <origin xyz="-1.286987800e-01 -1.604580800e-05 8.945601700e-01" />
+       <mass value="1.790000000e+01" />
+       <inertia ixx="1.009479700e+04" ixy="-3.568141800e-02" ixz="1.213165300e+03"
+       iyy="1.027057300e+04" iyz="7.021994000e-02"
+       izz="1.971602000e+02" />
+    </inertial>
   </link>
   <joint name="$(arg prefix)lift_fixed_joint" type="fixed">
@@ -68,26 +75,9 @@
   </xacro:ffw_follower_body>
   <xacro:rh_p12_rn_a parent="$(arg prefix)arm_l_link7" prefix="$(arg prefix)gripper_l_">
-    <origin xyz="0 0 -0.078" rpy="0 3.14159265359 0"/>
+    <origin xyz="0 0 -0.078" rpy="0 3.14159265359 3.14159265359"/>
   </xacro:rh_p12_rn_a>
   <xacro:rh_p12_rn_a parent="$(arg prefix)arm_r_link7" prefix="$(arg prefix)gripper_r_">
-    <origin xyz="0 0 -0.078" rpy="0 3.14159265359 0"/>
+    <origin xyz="0 0 -0.078" rpy="0 3.14159265359 3.14159265359"/>
   </xacro:rh_p12_rn_a>
-  <link name="$(arg prefix)left_wheel_steer_link">
-    <visual>
-      <origin xyz="0 0 0" rpy="0 0 0" />
-      <geometry>
-        <mesh filename="${meshes_file_direction}/left_wheel_steer_link.stl" scale="0.001 0.001 0.001" />
-      </geometry>
-      <material name="silver">
-        <color rgba="0.75 0.75 0.75 1"/>
-      </material>
-    </visual>
-    <collision>
-      <origin xyz="0 0 0" rpy="0 0 0" />
-      <geometry>
-        <mesh filename="${meshes_file_direction}/left_wheel_steer_link.stl" scale="0.001 0.001 0.001" />
-      </geometry>
-    </collision>
-  </link>
   <joint name="$(arg prefix)left_wheel_steer" type="revolute">
       <parent link="$(arg prefix)base_link"/>
@@ -97,4 +87,28 @@
       <limit velocity="4.8" effort="1" lower="${-pi*6.0}" upper="${pi*6.0}" />
   </joint>
+  <link name="$(arg prefix)left_wheel_steer_link">
+    <visual>
+      <origin xyz="0 0 0" rpy="0 0 0" />
+      <geometry>
+        <mesh filename="${meshes_file_direction}/left_wheel_steer_link.stl" scale="0.001 0.001 0.001" />
+      </geometry>
+      <material name="silver">
+        <color rgba="0.75 0.75 0.75 1"/>
+      </material>
+    </visual>
+    <collision>
+      <origin xyz="0 0 0" rpy="0 0 0" />
+      <geometry>
+        <mesh filename="${meshes_file_direction}/left_wheel_steer_link.stl" scale="0.001 0.001 0.001" />
+      </geometry>
+    </collision>
+    <inertial>
+       <origin xyz="9.802769300e-03 -5.471240900e-02 -1.376533800e-01" />
+       <mass value="7.550951000e-01" />
+       <inertia ixx="2.797326600e-03" ixy="-3.290807800e-05" ixz="-1.950671800e-04"
+       iyy="3.582264900e-03" iyz="-2.853290700e-04"
+       izz="1.683594000e-03" />
+    </inertial>
+  </link>
   <joint name="$(arg prefix)left_wheel_drive" type="revolute">
       <parent link="$(arg prefix)left_wheel_steer_link"/>
@@ -120,4 +134,11 @@
       </geometry>
     </collision>
+    <inertial>
+       <origin xyz="0.000000000e+00 -1.499601700e-03 0.000000000e+00" />
+       <mass value="3.795460500e+00" />
+       <inertia ixx="7.187881500e-03" ixy="0.000000000e+00" ixz="0.000000000e+00"
+       iyy="1.156399900e-02" iyz="0.000000000e+00"
+       izz="7.187977000e-03" />
+    </inertial>
   </link>
   <joint name="$(arg prefix)right_wheel_steer" type="revolute">
@@ -144,4 +165,11 @@
       </geometry>
     </collision>
+    <inertial>
+       <origin xyz="9.802728600e-03 5.471240900e-02 -1.376533400e-01" />
+       <mass value="7.550951000e-01" />
+       <inertia ixx="2.797322900e-03" ixy="3.290833300e-05" ixz="-1.950642500e-04"
+       iyy="3.582262300e-03" iyz="2.853288400e-04"
+       izz="1.683595100e-03" />
+    </inertial>
   </link>
   <joint name="$(arg prefix)right_wheel_drive" type="revolute">
@@ -168,4 +196,11 @@
       </geometry>
     </collision>
+    <inertial>
+       <origin xyz="0.000000000e+00 1.499601700e-03 0.000000000e+00" />
+       <mass value="3.795460500e+00" />
+       <inertia ixx="7.187881500e-03" ixy="0.000000000e+00" ixz="0.000000000e+00"
+       iyy="1.156399900e-02" iyz="0.000000000e+00"
+       izz="7.187977000e-03" />
+    </inertial>
   </link>
   <joint name="$(arg prefix)rear_wheel_steer" type="revolute">
@@ -192,4 +227,11 @@
       </geometry>
     </collision>
+    <inertial>
+       <origin xyz="9.802728600e-03 5.471240900e-02 -1.376533400e-01" />
+       <mass value="7.550951000e-01" />
+       <inertia ixx="2.797322900e-03" ixy="3.290833300e-05" ixz="-1.950642500e-04"
+       iyy="3.582262300e-03" iyz="2.853288400e-04"
+       izz="1.683595100e-03" />
+    </inertial>
   </link>
   <joint name="$(arg prefix)rear_wheel_drive" type="revolute">
@@ -216,4 +258,11 @@
       </geometry>
     </collision>
+    <inertial>
+       <origin xyz="0.000000000e+00 1.499601700e-03 0.000000000e+00" />
+       <mass value="3.795460500e+00" />
+       <inertia ixx="7.187881500e-03" ixy="0.000000000e+00" ixz="0.000000000e+00"
+       iyy="1.156399900e-02" iyz="0.000000000e+00"
+       izz="7.187977000e-03" />
+    </inertial>
   </link>
   <xacro:ffw_sg2_follower_system
