Commit message: Revert "Merge branch 'feature-dockerfile' of github.com:ROBOTIS-GIT/ai_worker into feature-trigger"
This reverts commit 301820ad83d1060e7a058c1f385c32059319f0cc, reversing
changes made to 22f69666624d58d964572e41ae1e680ee989843a.

File: ffw_description/urdf/ffw_bg2_rev2_follower/ffw_bg2_follower.urdf.xacro (robot description, xacro)
@@ -43,8 +43,8 @@
   </xacro:ffw_follower_body>
   <xacro:rh_p12_rn_a parent="$(arg prefix)arm_l_link7" prefix="$(arg prefix)gripper_l_">
-    <origin xyz="0 0 -0.05" rpy="0 3.14159265359 3.14159265359"/>
+    <origin xyz="0 0 -0.05" rpy="0 3.14159265359 0"/>
   </xacro:rh_p12_rn_a>
   <xacro:rh_p12_rn_a parent="$(arg prefix)arm_r_link7" prefix="$(arg prefix)gripper_r_">
-    <origin xyz="0 0 -0.05" rpy="0 3.14159265359 3.14159265359"/>
+    <origin xyz="0 0 -0.05" rpy="0 3.14159265359 0"/>
   </xacro:rh_p12_rn_a>
   <xacro:ffw_bg2_follower_system

File: ffw_description/urdf/ffw_bg2_rev3_follower/ffw_bg2_follower.urdf.xacro (robot description, xacro)
@@ -43,8 +43,8 @@
   </xacro:ffw_follower_body>
   <xacro:rh_p12_rn_a parent="$(arg prefix)arm_l_link7" prefix="$(arg prefix)gripper_l_">
-    <origin xyz="0 0 -0.05" rpy="0 3.14159265359 3.14159265359"/>
+    <origin xyz="0 0 -0.05" rpy="0 3.14159265359 0"/>
   </xacro:rh_p12_rn_a>
   <xacro:rh_p12_rn_a parent="$(arg prefix)arm_r_link7" prefix="$(arg prefix)gripper_r_">
-    <origin xyz="0 0 -0.05" rpy="0 3.14159265359 3.14159265359"/>
+    <origin xyz="0 0 -0.05" rpy="0 3.14159265359 0"/>
   </xacro:rh_p12_rn_a>
   <xacro:ffw_bg2_follower_system

File: ffw_description/urdf/ffw_bg2_rev4_follower/ffw_bg2_follower.urdf.xacro (robot description, xacro)
@@ -45,8 +45,8 @@
   </xacro:ffw_follower_body>
   <xacro:rh_p12_rn_a parent="$(arg prefix)arm_l_link7" prefix="$(arg prefix)gripper_l_">
-    <origin xyz="0 0 -0.078" rpy="0 3.14159265359 3.14159265359"/>
+    <origin xyz="0 0 -0.078" rpy="0 3.14159265359 0"/>
   </xacro:rh_p12_rn_a>
   <xacro:rh_p12_rn_a parent="$(arg prefix)arm_r_link7" prefix="$(arg prefix)gripper_r_">
-    <origin xyz="0 0 -0.078" rpy="0 3.14159265359 3.14159265359"/>
+    <origin xyz="0 0 -0.078" rpy="0 3.14159265359 0"/>
   </xacro:rh_p12_rn_a>
   <xacro:ffw_bg2_follower_system
